File: Kicad Files/shematic1/shematic1.kicad_pcb (KiCad board)
At the start: 4 copper layers, 246.5 x 189.2 mm, 418 parts

Commit message: updated pcb
Parts:
- added ?: , , F.Cu at (124.2, 93.5)
- added ?: , , F.Cu at (124.2, 51.3)
- added REF**: C_0603_1608Metric, Capacitor_SMD:C_0603_1608Metric, F.Cu at (73.2, 71.8)
- added REF**: C_0603_1608Metric, Capacitor_SMD:C_0603_1608Metric, F.Cu at (73.5, 155.5)
- added REF**: C_0603_1608Metric, Capacitor_SMD:C_0603_1608Metric, F.Cu at (73.5, 176.5)
- added REF**: C_0603_1608Metric, Capacitor_SMD:C_0603_1608Metric, F.Cu at (83.8, 113.5)
- added REF**: C_0603_1608Metric, Capacitor_SMD:C_0603_1608Metric, F.Cu at (20.2, 176.5)
- added REF**: C_0603_1608Metric, Capacitor_SMD:C_0603_1608Metric, F.Cu at (104.5, 92.8)
- added REF**: TerminalBlock_MaiXu_MX126-5.0-02P_1x02_P5.00mm, TerminalBlock:TerminalBlock_MaiXu_MX126-5.0-02P_1x02_P5.00mm, F.Cu at (259.0, 24.0)
- added REF**: C_0603_1608Metric, Capacitor_SMD:C_0603_1608Metric, F.Cu at (115.0, 50.5)
- added REF**: C_0603_1608Metric, Capacitor_SMD:C_0603_1608Metric, F.Cu at (20.2, 71.8)
- added REF**: C_0603_1608Metric, Capacitor_SMD:C_0603_1608Metric, F.Cu at (31.0, 92.8)
- added REF**: C_0603_1608Metric, Capacitor_SMD:C_0603_1608Metric, F.Cu at (178.2, 155.5)
- added REF**: C_0603_1608Metric, Capacitor_SMD:C_0603_1608Metric, F.Cu at (62.5, 71.8)
- added REF**: C_0603_1608Metric, Capacitor_SMD:C_0603_1608Metric, F.Cu at (45.8, 82.5)
- added REF**: C_0603_1608Metric, Capacitor_SMD:C_0603_1608Metric, F.Cu at (20.2, 92.8)
- added REF**: C_0603_1608Metric, Capacitor_SMD:C_0603_1608Metric, F.Cu at (94.2, 155.5)
- added REF**: C_0603_1608Metric, Capacitor_SMD:C_0603_1608Metric, F.Cu at (157.2, 92.8)
- added REF**: C_0603_1608Metric, Capacitor_SMD:C_0603_1608Metric, F.Cu at (31.2, 155.5)
- added REF**: C_0603_1608Metric, Capacitor_SMD:C_0603_1608Metric, F.Cu at (41.8, 176.5)
- added REF**: C_0603_1608Metric, Capacitor_SMD:C_0603_1608Metric, F.Cu at (136.2, 176.5)
- added REF**: C_0603_1608Metric, Capacitor_SMD:C_0603_1608Metric, F.Cu at (167.8, 50.5)
- added REF**: C_0603_1608Metric, Capacitor_SMD:C_0603_1608Metric, F.Cu at (20.2, 134.5)
- added REF**: C_0603_1608Metric, Capacitor_SMD:C_0603_1608Metric, F.Cu at (136.2, 155.5)
- added REF**: C_0603_1608Metric, Capacitor_SMD:C_0603_1608Metric, F.Cu at (31.0, 71.8)
- added REF**: C_0603_1608Metric, Capacitor_SMD:C_0603_1608Metric, F.Cu at (168.0, 155.5)
- added REF**: C_0603_1608Metric, Capacitor_SMD:C_0603_1608Metric, F.Cu at (73.2, 134.5)
- added REF**: C_0603_1608Metric, Capacitor_SMD:C_0603_1608Metric, F.Cu at (52.0, 134.5)
- added REF**: C_0603_1608Metric, Capacitor_SMD:C_0603_1608Metric, F.Cu at (167.8, 92.8)
- added REF**: C_0603_1608Metric, Capacitor_SMD:C_0603_1608Metric, F.Cu at (41.5, 113.5)
- added REF**: C_0603_1608Metric, Capacitor_SMD:C_0603_1608Metric, F.Cu at (125.8, 71.8)
- added REF**: C_0603_1608Metric, Capacitor_SMD:C_0603_1608Metric, F.Cu at (146.5, 113.5)
- added REF**: C_0603_1608Metric, Capacitor_SMD:C_0603_1608Metric, F.Cu at (178.2, 176.5)
- added REF**: C_0603_1608Metric, Capacitor_SMD:C_0603_1608Metric, F.Cu at (104.8, 176.5)
- added REF**: C_0603_1608Metric, Capacitor_SMD:C_0603_1608Metric, F.Cu at (41.5, 71.8)
- added REF**: C_0603_1608Metric, Capacitor_SMD:C_0603_1608Metric, F.Cu at (126.0, 155.5)
- added REF**: C_0603_1608Metric, Capacitor_SMD:C_0603_1608Metric, F.Cu at (178.0, 71.8)
- added REF**: C_0603_1608Metric, Capacitor_SMD:C_0603_1608Metric, F.Cu at (109.0, 82.5)
- added REF**: C_0603_1608Metric, Capacitor_SMD:C_0603_1608Metric, F.Cu at (41.5, 50.5)
- added REF**: C_0603_1608Metric, Capacitor_SMD:C_0603_1608Metric, F.Cu at (41.5, 92.8)
- added REF**: C_0603_1608Metric, Capacitor_SMD:C_0603_1608Metric, F.Cu at (41.5, 134.5)
- added REF**: C_0603_1608Metric, Capacitor_SMD:C_0603_1608Metric, F.Cu at (45.8, 40.2)
- added REF**: C_0603_1608Metric, Capacitor_SMD:C_0603_1608Metric, F.Cu at (129.8, 82.5)
- added REF**: C_0603_1608Metric, Capacitor_SMD:C_0603_1608Metric, F.Cu at (115.0, 113.5)
- added REF**: C_0603_1608Metric, Capacitor_SMD:C_0603_1608Metric, F.Cu at (157.2, 29.8)
- added REF**: C_0603_1608Metric, Capacitor_SMD:C_0603_1608Metric, F.Cu at (125.8, 92.8)
- added REF**: C_0603_1608Metric, Capacitor_SMD:C_0603_1608Metric, F.Cu at (31.0, 113.5)
- added REF**: C_0603_1608Metric, Capacitor_SMD:C_0603_1608Metric, F.Cu at (83.8, 50.5)
- added REF**: C_0603_1608Metric, Capacitor_SMD:C_0603_1608Metric, F.Cu at (157.5, 155.5)
- added REF**: C_0603_1608Metric, Capacitor_SMD:C_0603_1608Metric, F.Cu at (146.5, 92.8)
- added REF**: C_0603_1608Metric, Capacitor_SMD:C_0603_1608Metric, F.Cu at (94.0, 29.8)
- added REF**: C_0603_1608Metric, Capacitor_SMD:C_0603_1608Metric, F.Cu at (146.5, 134.5)
- added REF**: C_0603_1608Metric, Capacitor_SMD:C_0603_1608Metric, F.Cu at (31.0, 29.8)
- added REF**: C_0603_1608Metric, Capacitor_SMD:C_0603_1608Metric, F.Cu at (52.0, 29.8)
- added REF**: C_0603_1608Metric, Capacitor_SMD:C_0603_1608Metric, F.Cu at (188.8, 29.8)
- added REF**: C_0603_1608Metric, Capacitor_SMD:C_0603_1608Metric, F.Cu at (136.0, 71.8)
- added REF**: C_0603_1608Metric, Capacitor_SMD:C_0603_1608Metric, F.Cu at (62.5, 134.5)
- added REF**: C_0603_1608Metric, Capacitor_SMD:C_0603_1608Metric, F.Cu at (129.8, 40.2)
- added REF**: C_0603_1608Metric, Capacitor_SMD:C_0603_1608Metric, F.Cu at (67.0, 124.2)
- added REF**: C_0603_1608Metric, Capacitor_SMD:C_0603_1608Metric, F.Cu at (20.2, 29.8)
- added REF**: C_0603_1608Metric, Capacitor_SMD:C_0603_1608Metric, F.Cu at (52.0, 113.5)
- added REF**: C_0603_1608Metric, Capacitor_SMD:C_0603_1608Metric, F.Cu at (20.2, 113.5)
- added REF**: C_0603_1608Metric, Capacitor_SMD:C_0603_1608Metric, F.Cu at (104.5, 29.8)
- added REF**: C_0603_1608Metric, Capacitor_SMD:C_0603_1608Metric, F.Cu at (41.5, 29.8)
- added REF**: C_0603_1608Metric, Capacitor_SMD:C_0603_1608Metric, F.Cu at (188.8, 113.5)
- added REF**: C_0603_1608Metric, Capacitor_SMD:C_0603_1608Metric, F.Cu at (83.8, 71.8)
- added REF**: C_0603_1608Metric, Capacitor_SMD:C_0603_1608Metric, F.Cu at (167.8, 71.8)
- added REF**: C_0603_1608Metric, Capacitor_SMD:C_0603_1608Metric, F.Cu at (46.2, 166.2)
- added REF**: C_0603_1608Metric, Capacitor_SMD:C_0603_1608Metric, F.Cu at (52.2, 176.5)
- added REF**: C_0603_1608Metric, Capacitor_SMD:C_0603_1608Metric, F.Cu at (104.5, 134.5)
- added REF**: C_0603_1608Metric, Capacitor_SMD:C_0603_1608Metric, F.Cu at (172.0, 124.2)
- added REF**: C_0603_1608Metric, Capacitor_SMD:C_0603_1608Metric, F.Cu at (25.0, 124.2)
- added REF**: C_0603_1608Metric, Capacitor_SMD:C_0603_1608Metric, F.Cu at (73.2, 50.5)
- added REF**: C_0603_1608Metric, Capacitor_SMD:C_0603_1608Metric, F.Cu at (125.8, 113.5)
- added REF**: C_0603_1608Metric, Capacitor_SMD:C_0603_1608Metric, F.Cu at (188.8, 92.8)
- added REF**: C_0603_1608Metric, Capacitor_SMD:C_0603_1608Metric, F.Cu at (20.2, 155.5)
- added REF**: C_0603_1608Metric, Capacitor_SMD:C_0603_1608Metric, F.Cu at (84.0, 176.5)
- added REF**: C_0603_1608Metric, Capacitor_SMD:C_0603_1608Metric, F.Cu at (178.0, 113.5)
- added REF**: C_0603_1608Metric, Capacitor_SMD:C_0603_1608Metric, F.Cu at (104.8, 155.5)
- added REF**: C_0603_1608Metric, Capacitor_SMD:C_0603_1608Metric, F.Cu at (109.0, 124.2)
- added REF**: C_0603_1608Metric, Capacitor_SMD:C_0603_1608Metric, F.Cu at (146.8, 155.5)
- added REF**: C_0603_1608Metric, Capacitor_SMD:C_0603_1608Metric, F.Cu at (83.8, 29.8)
- added REF**: C_0603_1608Metric, Capacitor_SMD:C_0603_1608Metric, F.Cu at (167.8, 134.5)
- added REF**: C_0603_1608Metric, Capacitor_SMD:C_0603_1608Metric, F.Cu at (136.0, 134.5)
- added REF**: C_0603_1608Metric, Capacitor_SMD:C_0603_1608Metric, F.Cu at (115.0, 29.8)
- added REF**: C_0603_1608Metric, Capacitor_SMD:C_0603_1608Metric, F.Cu at (52.0, 92.8)
- added REF**: C_0603_1608Metric, Capacitor_SMD:C_0603_1608Metric, F.Cu at (94.2, 176.5)
- added REF**: C_0603_1608Metric, Capacitor_SMD:C_0603_1608Metric, F.Cu at (62.5, 92.8)
- added REF**: C_0603_1608Metric, Capacitor_SMD:C_0603_1608Metric, F.Cu at (25.0, 82.5)
- added REF**: C_0603_1608Metric, Capacitor_SMD:C_0603_1608Metric, F.Cu at (168.0, 176.5)
- added REF**: C_0603_1608Metric, Capacitor_SMD:C_0603_1608Metric, F.Cu at (88.0, 82.5)
- added REF**: C_0603_1608Metric, Capacitor_SMD:C_0603_1608Metric, F.Cu at (129.8, 124.2)
- added REF**: C_0603_1608Metric, Capacitor_SMD:C_0603_1608Metric, F.Cu at (67.0, 40.2)
- added REF**: C_0603_1608Metric, Capacitor_SMD:C_0603_1608Metric, F.Cu at (73.2, 113.5)
- added REF**: C_0603_1608Metric, Capacitor_SMD:C_0603_1608Metric, F.Cu at (125.8, 50.5)
- added REF**: C_0603_1608Metric, Capacitor_SMD:C_0603_1608Metric, F.Cu at (157.2, 71.8)
- added REF**: C_0603_1608Metric, Capacitor_SMD:C_0603_1608Metric, F.Cu at (151.2, 166.2)
- added REF**: C_0603_1608Metric, Capacitor_SMD:C_0603_1608Metric, F.Cu at (62.5, 113.5)
- added REF**: C_0603_1608Metric, Capacitor_SMD:C_0603_1608Metric, F.Cu at (136.0, 29.8)
- added REF**: C_0603_1608Metric, Capacitor_SMD:C_0603_1608Metric, F.Cu at (178.0, 134.5)
- added REF**: C_0603_1608Metric, Capacitor_SMD:C_0603_1608Metric, F.Cu at (52.0, 71.8)
- added REF**: C_0603_1608Metric, Capacitor_SMD:C_0603_1608Metric, F.Cu at (67.2, 166.2)
- added REF**: C_0603_1608Metric, Capacitor_SMD:C_0603_1608Metric, F.Cu at (109.2, 166.2)
- added REF**: C_0603_1608Metric, Capacitor_SMD:C_0603_1608Metric, F.Cu at (62.8, 155.5)
- added REF**: C_0603_1608Metric, Capacitor_SMD:C_0603_1608Metric, F.Cu at (94.0, 134.5)
- added REF**: C_0603_1608Metric, Capacitor_SMD:C_0603_1608Metric, F.Cu at (130.0, 166.2)
- added REF**: C_0603_1608Metric, Capacitor_SMD:C_0603_1608Metric, F.Cu at (45.8, 124.2)
- added REF**: C_0603_1608Metric, Capacitor_SMD:C_0603_1608Metric, F.Cu at (94.0, 50.5)
- added REF**: C_0603_1608Metric, Capacitor_SMD:C_0603_1608Metric, F.Cu at (146.5, 71.8)
- added REF**: C_0603_1608Metric, Capacitor_SMD:C_0603_1608Metric, F.Cu at (115.0, 92.8)
- added REF**: C_0603_1608Metric, Capacitor_SMD:C_0603_1608Metric, F.Cu at (178.0, 29.8)
- added REF**: C_0603_1608Metric, Capacitor_SMD:C_0603_1608Metric, F.Cu at (188.8, 134.5)
- added REF**: C_0603_1608Metric, Capacitor_SMD:C_0603_1608Metric, F.Cu at (88.2, 166.2)
- added REF**: C_0603_1608Metric, Capacitor_SMD:C_0603_1608Metric, F.Cu at (188.8, 50.5)
- added REF**: C_0603_1608Metric, Capacitor_SMD:C_0603_1608Metric, F.Cu at (104.5, 71.8)
- added REF**: C_0603_1608Metric, Capacitor_SMD:C_0603_1608Metric, F.Cu at (62.5, 50.5)
- added REF**: C_0603_1608Metric, Capacitor_SMD:C_0603_1608Metric, F.Cu at (136.0, 113.5)
- added REF**: C_0603_1608Metric, Capacitor_SMD:C_0603_1608Metric, F.Cu at (104.5, 113.5)
- added REF**: C_0603_1608Metric, Capacitor_SMD:C_0603_1608Metric, F.Cu at (188.8, 71.8)
- added REF**: C_0603_1608Metric, Capacitor_SMD:C_0603_1608Metric, F.Cu at (146.5, 29.8)
- added REF**: C_0603_1608Metric, Capacitor_SMD:C_0603_1608Metric, F.Cu at (62.8, 176.5)
- added REF**: C_0603_1608Metric, Capacitor_SMD:C_0603_1608Metric, F.Cu at (167.8, 113.5)
- added REF**: C_0603_1608Metric, Capacitor_SMD:C_0603_1608Metric, F.Cu at (172.0, 40.2)
- added REF**: C_0603_1608Metric, Capacitor_SMD:C_0603_1608Metric, F.Cu at (20.2, 50.5)
- added REF**: C_0603_1608Metric, Capacitor_SMD:C_0603_1608Metric, F.Cu at (83.8, 134.5)
- added REF**: C_0603_1608Metric, Capacitor_SMD:C_0603_1608Metric, F.Cu at (157.2, 50.5)
- added REF**: C_0603_1608Metric, Capacitor_SMD:C_0603_1608Metric, F.Cu at (83.8, 92.8)
- added REF**: C_0603_1608Metric, Capacitor_SMD:C_0603_1608Metric, F.Cu at (178.0, 50.5)
- added REF**: C_0603_1608Metric, Capacitor_SMD:C_0603_1608Metric, F.Cu at (108.8, 40.2)
- added REF**: C_0603_1608Metric, Capacitor_SMD:C_0603_1608Metric, F.Cu at (189.0, 176.5)
- added REF**: C_0603_1608Metric, Capacitor_SMD:C_0603_1608Metric, F.Cu at (172.0, 82.5)
- added REF**: C_0603_1608Metric, Capacitor_SMD:C_0603_1608Metric, F.Cu at (115.2, 176.5)
- added REF**: C_0603_1608Metric, Capacitor_SMD:C_0603_1608Metric, F.Cu at (125.8, 134.5)
- added REF**: C_0603_1608Metric, Capacitor_SMD:C_0603_1608Metric, F.Cu at (73.2, 29.8)
- added REF**: C_0603_1608Metric, Capacitor_SMD:C_0603_1608Metric, F.Cu at (94.0, 113.5)
- added REF**: C_0603_1608Metric, Capacitor_SMD:C_0603_1608Metric, F.Cu at (67.0, 82.5)
- added REF**: C_0603_1608Metric, Capacitor_SMD:C_0603_1608Metric, F.Cu at (157.5, 176.5)
- added REF**: C_0603_1608Metric, Capacitor_SMD:C_0603_1608Metric, F.Cu at (52.0, 50.5)
- added REF**: C_0603_1608Metric, Capacitor_SMD:C_0603_1608Metric, F.Cu at (115.2, 155.5)
- added REF**: C_0603_1608Metric, Capacitor_SMD:C_0603_1608Metric, F.Cu at (146.8, 176.5)
- added REF**: C_0603_1608Metric, Capacitor_SMD:C_0603_1608Metric, F.Cu at (94.0, 71.8)
- added REF**: C_0603_1608Metric, Capacitor_SMD:C_0603_1608Metric, F.Cu at (167.8, 29.8)
- added REF**: C_0603_1608Metric, Capacitor_SMD:C_0603_1608Metric, F.Cu at (178.0, 92.8)
- added REF**: C_0603_1608Metric, Capacitor_SMD:C_0603_1608Metric, F.Cu at (151.0, 40.2)
- added REF**: C_0603_1608Metric, Capacitor_SMD:C_0603_1608Metric, F.Cu at (157.2, 134.5)
- added REF**: C_0603_1608Metric, Capacitor_SMD:C_0603_1608Metric, F.Cu at (146.5, 50.5)
- added REF**: C_0603_1608Metric, Capacitor_SMD:C_0603_1608Metric, F.Cu at (151.0, 82.5)
- added REF**: C_0603_1608Metric, Capacitor_SMD:C_0603_1608Metric, F.Cu at (41.8, 155.5)
- added REF**: C_0603_1608Metric, Capacitor_SMD:C_0603_1608Metric, F.Cu at (88.0, 124.2)
- added REF**: C_0603_1608Metric, Capacitor_SMD:C_0603_1608Metric, F.Cu at (151.0, 124.2)
- added REF**: C_0603_1608Metric, Capacitor_SMD:C_0603_1608Metric, F.Cu at (189.0, 155.5)
- added REF**: C_0603_1608Metric, Capacitor_SMD:C_0603_1608Metric, F.Cu at (157.2, 113.5)
- added REF**: C_0603_1608Metric, Capacitor_SMD:C_0603_1608Metric, F.Cu at (31.0, 50.5)
- added REF**: C_0603_1608Metric, Capacitor_SMD:C_0603_1608Metric, F.Cu at (52.2, 155.5)
- added REF**: C_0603_1608Metric, Capacitor_SMD:C_0603_1608Metric, F.Cu at (25.2, 166.2)
- added REF**: C_0603_1608Metric, Capacitor_SMD:C_0603_1608Metric, F.Cu at (115.0, 71.8)
- added REF**: C_0603_1608Metric, Capacitor_SMD:C_0603_1608Metric, F.Cu at (73.2, 92.8)
- added REF**: C_0603_1608Metric, Capacitor_SMD:C_0603_1608Metric, F.Cu at (125.8, 29.8)
- added REF**: C_0603_1608Metric, Capacitor_SMD:C_0603_1608Metric, F.Cu at (126.0, 176.5)
- added REF**: C_0603_1608Metric, Capacitor_SMD:C_0603_1608Metric, F.Cu at (84.0, 155.5)
- added REF**: C_0603_1608Metric, Capacitor_SMD:C_0603_1608Metric, F.Cu at (172.2, 166.2)
- added REF**: C_0603_1608Metric, Capacitor_SMD:C_0603_1608Metric, F.Cu at (62.5, 29.8)
- added REF**: C_0603_1608Metric, Capacitor_SMD:C_0603_1608Metric, F.Cu at (94.0, 92.8)
- added REF**: C_0603_1608Metric, Capacitor_SMD:C_0603_1608Metric, F.Cu at (136.0, 92.8)
- added REF**: C_0603_1608Metric, Capacitor_SMD:C_0603_1608Metric, F.Cu at (104.5, 50.5)
- added REF**: C_0603_1608Metric, Capacitor_SMD:C_0603_1608Metric, F.Cu at (88.0, 40.2)
- added REF**: C_0603_1608Metric, Capacitor_SMD:C_0603_1608Metric, F.Cu at (24.8, 40.2)
- added REF**: C_0603_1608Metric, Capacitor_SMD:C_0603_1608Metric, F.Cu at (136.0, 50.5)
- added REF**: C_0603_1608Metric, Capacitor_SMD:C_0603_1608Metric, F.Cu at (31.0, 134.5)
- added REF**: C_0603_1608Metric, Capacitor_SMD:C_0603_1608Metric, F.Cu at (115.0, 134.5)
- added REF**: C_0603_1608Metric, Capacitor_SMD:C_0603_1608Metric, F.Cu at (31.2, 176.5)
- moved REF** 54.1 mm to (258.8, 100.4), turned to 0 degrees
Routing:
- net (no net): track 2530.5 -> 11383.3 mm, vias 96 -> 428
