File: hardware/KiCad/shematic1/shematic1.kicad_pcb (KiCad board)
At the start: 4 copper layers, 246.5 x 189.2 mm, 589 parts

Commit message: fix compilation in linux
Parts:
- removed ? (x2): , 
- removed the REF** at (73.2, 71.8)
- removed the REF** at (57.2, 108.5)
- removed the REF** at (73.5, 155.5)
- removed the REF** at (109.7, 182.0)
- removed the REF** at (73.5, 176.5)
- removed the REF** at (183.2, 98.0)
- removed the REF** at (83.8, 113.5)
- removed the REF** at (20.2, 176.5)
- removed the REF** at (104.5, 92.8)
- removed the REF** at (115.0, 50.5)
- removed the REF** at (151.7, 182.0)
- removed the REF** at (172.7, 77.0)
- removed the REF** at (109.7, 140.0)
- removed the REF** at (20.2, 71.8)
- removed the REF** at (46.7, 45.5)
- removed the REF** at (172.7, 161.0)
- removed the REF** at (151.7, 108.5)
- removed the REF** at (36.2, 108.5)
- removed the REF** at (31.0, 92.8)
- removed the REF** at (25.7, 45.5)
- removed the REF** at (67.7, 161.0)
- removed the REF** at (178.2, 155.5)
- removed the REF** at (130.7, 24.5)
- removed the REF** at (78.2, 98.0)
- removed the REF** at (151.7, 150.5)
- removed the REF** at (99.2, 45.5)
- removed the REF** at (62.5, 71.8)
- removed the REF** at (57.2, 150.5)
- removed the REF** at (45.8, 82.5)
- removed the REF** at (120.2, 182.0)
- removed the REF** at (20.2, 92.8)
- removed the REF** at (94.2, 155.5)
- removed the REF** at (25.7, 150.5)
- removed the REF** at (46.7, 140.0)
- removed the REF** at (151.7, 87.5)
- removed the REF** at (157.2, 92.8)
- removed the REF** at (36.2, 171.5)
- removed the REF** at (67.7, 171.5)
- removed the REF** at (31.2, 155.5)
- removed the REF** at (41.8, 176.5)
- removed the REF** at (46.7, 77.0)
- removed the REF** at (136.2, 176.5)
- removed the REF** at (167.8, 50.5)
- removed the REF** at (20.2, 134.5)
- removed the REF** at (136.2, 155.5)
- removed the REF** at (31.0, 71.8)
- removed the REF** at (109.7, 98.0)
- removed the REF** at (57.2, 161.0)
- removed the REF** at (57.2, 77.0)
- removed the REF** at (151.7, 56.0)
- removed the REF** at (168.0, 155.5)
- removed the REF** at (172.7, 108.5)
- removed the REF** at (172.7, 98.0)
- removed the REF** at (36.2, 119.0)
- removed the REF** at (73.2, 134.5)
- removed the REF** at (36.2, 129.5)
- removed the REF** at (52.0, 134.5)
- removed the REF** at (46.7, 87.5)
- removed the REF** at (167.8, 92.8)
- removed the REF** at (109.7, 45.5)
- removed the REF** at (109.7, 129.5)
- removed the REF** at (57.2, 87.5)
- removed the REF** at (57.2, 45.5)
- removed the REF** at (78.2, 24.5)
- removed the REF** at (151.7, 98.0)
- removed the REF** at (120.2, 129.5)
- removed the REF** at (151.7, 77.0)
- removed the REF** at (41.5, 113.5)
- removed the REF** at (120.2, 45.5)
- removed the REF** at (67.7, 66.5)
- removed the REF** at (88.7, 56.0)
- removed the REF** at (125.8, 71.8)
- removed the REF** at (109.7, 87.5)
- removed the REF** at (162.2, 77.0)
- removed the REF** at (151.7, 140.0)
- removed the REF** at (146.5, 113.5)
- removed the REF** at (67.7, 98.0)
- removed the REF** at (172.7, 150.5)
- removed the REF** at (46.7, 66.5)
- removed the REF** at (99.2, 98.0)
- removed the REF** at (183.2, 77.0)
- removed the REF** at (57.2, 24.5)
- removed the REF** at (178.2, 176.5)
- removed the REF** at (78.2, 129.5)
- removed the REF** at (120.2, 87.5)
- removed the REF** at (104.8, 176.5)
- removed the REF** at (99.2, 77.0)
- removed the REF** at (46.7, 56.0)
- removed the REF** at (41.5, 71.8)
- removed the REF** at (126.0, 155.5)
- removed the REF** at (99.2, 171.5)
- removed the REF** at (178.0, 71.8)
- removed the REF** at (109.0, 82.5)
- removed the REF** at (172.7, 140.0)
- removed the REF** at (141.2, 87.5)
- removed the REF** at (141.2, 98.0)
- removed the REF** at (141.2, 56.0)
- removed the REF** at (78.2, 140.0)
- removed the REF** at (41.5, 50.5)
- removed the REF** at (120.2, 140.0)
- removed the REF** at (41.5, 92.8)
- removed the REF** at (41.5, 134.5)
- removed the REF** at (25.7, 56.0)
- removed the REF** at (57.2, 140.0)
- removed the REF** at (25.7, 66.5)
- removed the REF** at (129.8, 82.5)
- removed the REF** at (115.0, 113.5)
- removed the REF** at (141.2, 77.0)
- removed the REF** at (125.8, 92.8)
- removed the REF** at (31.0, 113.5)
- removed the REF** at (83.8, 50.5)
- removed the REF** at (157.5, 155.5)
- removed the REF** at (78.2, 45.5)
- removed the REF** at (46.7, 24.5)
- removed the REF** at (36.2, 150.5)
- removed the REF** at (146.5, 92.8)
- removed the REF** at (88.7, 171.5)
- removed the REF** at (146.5, 134.5)
- removed the REF** at (162.2, 66.5)
- removed the REF** at (151.7, 24.5)
- removed the REF** at (136.0, 71.8)
- removed the REF** at (67.7, 24.5)
- removed the REF** at (62.5, 134.5)
- removed the REF** at (162.2, 98.0)
- removed the REF** at (162.2, 108.5)
- removed the REF** at (67.0, 124.2)
- removed the REF** at (25.7, 98.0)
- removed the REF** at (67.7, 77.0)
- removed the REF** at (141.2, 171.5)
- removed the REF** at (52.0, 113.5)
- removed the REF** at (88.7, 129.5)
- removed the REF** at (20.2, 113.5)
- removed the REF** at (130.7, 98.0)
- removed the REF** at (78.2, 87.5)
- removed the REF** at (99.2, 161.0)
- removed the REF** at (120.2, 161.0)
- removed the REF** at (188.8, 113.5)
- removed the REF** at (120.2, 77.0)
- removed the REF** at (83.8, 71.8)
- removed the REF** at (57.2, 119.0)
- removed the REF** at (183.2, 24.5)
- removed the REF** at (172.7, 24.5)
- removed the REF** at (167.8, 71.8)
- removed the REF** at (99.2, 182.0)
- removed the REF** at (162.2, 87.5)
- removed the REF** at (46.2, 166.2)
- removed the REF** at (46.7, 161.0)
- removed the REF** at (67.7, 108.5)
- removed the REF** at (52.2, 176.5)
- removed the REF** at (104.5, 134.5)
- removed the REF** at (162.2, 150.5)
- removed the REF** at (67.7, 129.5)
- removed the REF** at (172.0, 124.2)
- removed the REF** at (25.0, 124.2)
- removed the REF** at (88.7, 87.5)
- removed the REF** at (46.7, 129.5)
- removed the REF** at (151.7, 129.5)
- removed the REF** at (88.7, 24.5)
- removed the REF** at (25.7, 108.5)
- removed the REF** at (73.2, 50.5)
- removed the REF** at (125.8, 113.5)
- removed the REF** at (183.2, 171.5)
- removed the REF** at (109.7, 24.5)
- removed the REF** at (25.7, 140.0)
- removed the REF** at (99.2, 129.5)
- removed the REF** at (188.8, 92.8)
- removed the REF** at (172.7, 182.0)
- removed the REF** at (20.2, 155.5)
- removed the REF** at (84.0, 176.5)
- removed the REF** at (178.0, 113.5)
- removed the REF** at (151.7, 45.5)
- removed the REF** at (46.7, 150.5)
- removed the REF** at (25.7, 87.5)
- removed the REF** at (183.2, 87.5)
- removed the REF** at (183.2, 182.0)
- removed the REF** at (172.7, 66.5)
- removed the REF** at (67.7, 45.5)
- removed the REF** at (120.2, 108.5)
- removed the REF** at (78.2, 77.0)
- removed the REF** at (104.8, 155.5)
- removed the REF** at (109.0, 124.2)
- removed the REF** at (146.8, 155.5)
- removed the REF** at (167.8, 134.5)
- removed the REF** at (141.2, 66.5)
- removed the REF** at (88.7, 182.0)
- removed the REF** at (109.7, 66.5)
- removed the REF** at (120.2, 66.5)
- removed the REF** at (136.0, 134.5)
- removed the REF** at (151.7, 161.0)
- removed the REF** at (25.7, 129.5)
- removed the REF** at (151.7, 119.0)
- removed the REF** at (36.2, 87.5)
- removed the REF** at (141.2, 24.5)
- removed the REF** at (46.7, 171.5)
- removed the REF** at (52.0, 92.8)
- removed the REF** at (88.7, 45.5)
- removed the REF** at (94.2, 176.5)
- removed the REF** at (183.2, 108.5)
- removed the REF** at (99.2, 108.5)
- removed the REF** at (141.2, 119.0)
- removed the REF** at (36.2, 161.0)
- removed the REF** at (162.2, 161.0)
- removed the REF** at (120.2, 171.5)
- removed the REF** at (62.5, 92.8)
- removed the REF** at (25.0, 82.5)
- removed the REF** at (168.0, 176.5)
- removed the REF** at (57.2, 129.5)
- removed the REF** at (88.0, 82.5)
- removed the REF** at (130.7, 66.5)
- removed the REF** at (129.8, 124.2)
- removed the REF** at (36.2, 77.0)
- removed the REF** at (172.7, 87.5)
- removed the REF** at (73.2, 113.5)
- removed the REF** at (125.8, 50.5)
- removed the REF** at (141.2, 45.5)
- removed the REF** at (130.7, 129.5)
- removed the REF** at (57.2, 66.5)
- removed the REF** at (157.2, 71.8)
- removed the REF** at (151.2, 166.2)
- removed the REF** at (62.5, 113.5)
- removed the REF** at (151.7, 66.5)
- removed the REF** at (36.2, 182.0)
- removed the REF** at (88.7, 140.0)
- removed the REF** at (178.0, 134.5)
- removed the REF** at (52.0, 71.8)
- removed the REF** at (141.2, 129.5)
- removed the REF** at (130.7, 150.5)
- removed the REF** at (67.2, 166.2)
- removed the REF** at (109.2, 166.2)
- removed the REF** at (62.8, 155.5)
- removed the REF** at (46.7, 182.0)
- removed the REF** at (162.2, 182.0)
- removed the REF** at (88.7, 119.0)
- removed the REF** at (172.7, 171.5)
- removed the REF** at (78.2, 171.5)
- removed the REF** at (94.0, 134.5)
- removed the REF** at (78.2, 161.0)
- removed the REF** at (25.7, 24.5)
- removed the REF** at (130.0, 166.2)
- removed the REF** at (25.7, 161.0)
- removed the REF** at (45.8, 124.2)
- removed the REF** at (99.2, 150.5)
- removed the REF** at (120.2, 56.0)
- removed the REF** at (130.7, 140.0)
- removed the REF** at (94.0, 50.5)
- removed the REF** at (172.7, 129.5)
- removed the REF** at (146.5, 71.8)
- removed the REF** at (115.0, 92.8)
- removed the REF** at (183.2, 140.0)
- removed the REF** at (188.8, 134.5)
- removed the REF** at (88.2, 166.2)
- removed the REF** at (188.8, 50.5)
- removed the REF** at (104.5, 71.8)
- removed the REF** at (78.2, 119.0)
- removed the REF** at (99.2, 24.5)
- removed the REF** at (62.5, 50.5)
- removed the REF** at (162.2, 129.5)
- removed the REF** at (136.0, 113.5)
- removed the REF** at (172.7, 56.0)
- removed the REF** at (130.7, 87.5)
- removed the REF** at (104.5, 113.5)
- removed the REF** at (57.2, 56.0)
- removed the REF** at (188.8, 71.8)
- removed the REF** at (109.7, 56.0)
- removed the REF** at (67.7, 150.5)
- removed the REF** at (62.8, 176.5)
- removed the REF** at (183.2, 56.0)
- removed the REF** at (167.8, 113.5)
- removed the REF** at (88.7, 161.0)
- removed the REF** at (183.2, 129.5)
- removed the REF** at (130.7, 56.0)
- removed the REF** at (36.2, 66.5)
- removed the REF** at (130.7, 182.0)
- removed the REF** at (183.2, 119.0)
- removed the REF** at (20.2, 50.5)
- removed the REF** at (120.2, 150.5)
- removed the REF** at (83.8, 134.5)
- removed the REF** at (157.2, 50.5)
- removed the REF** at (67.7, 87.5)
- removed the REF** at (83.8, 92.8)
- removed the REF** at (78.2, 66.5)
- removed the REF** at (162.2, 45.5)
- removed the REF** at (109.7, 171.5)
- removed the REF** at (36.2, 56.0)
- removed the REF** at (99.2, 66.5)
- removed the REF** at (172.7, 119.0)
- removed the REF** at (25.7, 77.0)
- removed the REF** at (88.7, 66.5)
- removed the REF** at (178.0, 50.5)
- removed the REF** at (67.7, 119.0)
- removed the REF** at (151.7, 171.5)
- removed the REF** at (88.7, 150.5)
- removed the REF** at (189.0, 176.5)
- removed the REF** at (130.7, 77.0)
- removed the REF** at (183.2, 150.5)
- removed the REF** at (172.0, 82.5)
- removed the REF** at (115.2, 176.5)
- removed the REF** at (125.8, 134.5)
- removed the REF** at (109.7, 161.0)
- removed the REF** at (162.2, 140.0)
- removed the REF** at (46.7, 98.0)
- removed the REF** at (130.7, 119.0)
- removed the REF** at (94.0, 113.5)
- removed the REF** at (67.0, 82.5)
- removed the REF** at (157.5, 176.5)
- removed the REF** at (25.7, 119.0)
- removed the REF** at (52.0, 50.5)
- removed the REF** at (120.2, 24.5)
- removed the REF** at (172.7, 45.5)
- removed the REF** at (88.7, 77.0)
- removed the REF** at (115.2, 155.5)
- removed the REF** at (67.7, 140.0)
- removed the REF** at (146.8, 176.5)
- removed the REF** at (78.2, 150.5)
- removed the REF** at (94.0, 71.8)
- removed the REF** at (88.7, 108.5)
- removed the REF** at (99.2, 87.5)
- removed the REF** at (141.2, 161.0)
- removed the REF** at (178.0, 92.8)
- removed the REF** at (162.2, 171.5)
- removed the REF** at (120.2, 119.0)
- removed the REF** at (130.7, 161.0)
- removed the REF** at (57.2, 171.5)
- removed the REF** at (141.2, 140.0)
- removed the REF** at (130.7, 108.5)
- removed the REF** at (99.2, 56.0)
- removed the REF** at (157.2, 134.5)
- removed the REF** at (146.5, 50.5)
- removed the REF** at (130.7, 92.7)
- removed the REF** at (109.9, 176.5)
- removed the REF** at (141.1, 92.7)
- removed the REF** at (57.2, 182.0)
- removed the REF** at (99.4, 155.5)
- removed the REF** at (141.4, 176.5)
- removed the REF** at (99.2, 113.5)
- removed the REF** at (25.7, 134.5)
- removed the REF** at (130.9, 155.5)
- removed the REF** at (25.7, 71.7)
- removed the REF** at (162.2, 113.5)
- removed the REF** at (109.7, 113.5)
- removed the REF** at (88.8, 134.4)
- removed the REF** at (78.2, 182.0)
- removed the REF** at (46.9, 155.4)
- removed the REF** at (32.0, 166.2)
- removed the REF** at (67.7, 50.5)
- removed the REF** at (157.8, 124.3)
- removed the REF** at (183.4, 176.5)
- removed the REF** at (136.7, 124.3)
- removed the REF** at (46.9, 176.4)
- removed the REF** at (151.7, 50.5)
- removed the REF** at (78.2, 50.5)
- removed the REF** at (151.0, 82.5)
- removed the REF** at (162.2, 92.8)
- removed the REF** at (115.8, 82.5)
- removed the REF** at (141.1, 71.8)
- removed the REF** at (183.2, 134.5)
- removed the REF** at (130.6, 113.5)
- removed the REF** at (172.7, 113.5)
- removed the REF** at (120.4, 155.6)
- removed the REF** at (41.8, 155.5)
- removed the REF** at (57.4, 176.4)
- removed the REF** at (151.8, 92.8)
- removed the REF** at (25.9, 155.5)
- removed the REF** at (46.7, 92.7)
- removed the REF** at (183.4, 155.5)
- removed the REF** at (25.7, 92.7)
- removed the REF** at (152.0, 176.5)
- removed the REF** at (141.2, 182.0)
- removed the REF** at (57.1, 71.7)
- removed the REF** at (31.8, 82.5)
- removed the REF** at (88.7, 71.7)
- removed the REF** at (36.4, 155.5)
- removed the REF** at (74.1, 166.2)
- removed the REF** at (172.7, 71.7)
- removed the REF** at (157.8, 82.5)
- removed the REF** at (67.8, 71.7)
- removed the REF** at (120.2, 134.5)
- removed the REF** at (162.2, 56.0)
- removed the REF** at (162.2, 50.5)
- removed the REF** at (78.2, 113.5)
- removed the REF** at (179.0, 166.2)
- removed the REF** at (36.2, 134.5)
- removed the REF** at (46.6, 113.4)
- removed the REF** at (130.7, 134.5)
- removed the REF** at (141.1, 50.5)
- removed the REF** at (162.5, 155.5)
- removed the REF** at (99.2, 92.7)
- removed the REF** at (88.0, 124.2)
- removed the REF** at (68.0, 176.5)
- removed the REF** at (152.0, 155.5)
- removed the REF** at (99.2, 134.4)
- removed the REF** at (78.2, 134.5)
- removed the REF** at (78.2, 92.7)
- removed the REF** at (99.4, 176.4)
- removed the REF** at (172.8, 134.5)
- removed the REF** at (94.8, 124.2)
- removed the REF** at (172.8, 92.7)
- removed the REF** at (36.4, 176.5)
- removed the REF** at (162.2, 24.5)
- removed the REF** at (120.2, 98.0)
- removed the REF** at (136.7, 82.5)
- removed the REF** at (183.2, 71.8)
- removed the REF** at (78.2, 71.8)
- removed the REF** at (52.7, 124.2)
- removed the REF** at (25.7, 50.5)
- removed the REF** at (183.2, 92.7)
- removed the REF** at (57.1, 50.5)
- removed the REF** at (172.7, 50.5)
- removed the REF** at (36.2, 140.0)
- removed the REF** at (88.8, 92.7)
- removed the REF** at (172.9, 155.5)
- removed the REF** at (130.9, 176.5)
- removed the REF** at (141.1, 113.5)
- removed the REF** at (46.6, 71.7)
- removed the REF** at (57.1, 92.7)
- removed the REF** at (178.8, 124.2)
- removed the REF** at (162.2, 71.8)
- removed the REF** at (67.8, 134.5)
- removed the REF** at (151.0, 124.2)
- removed the REF** at (130.6, 71.7)
- removed the REF** at (36.2, 92.7)
- removed the REF** at (73.8, 82.5)
- removed the REF** at (52.9, 166.2)
- removed the REF** at (120.2, 113.6)
- removed the REF** at (46.7, 134.4)
- removed the REF** at (151.8, 134.5)
- removed the REF** at (141.2, 108.5)
- removed the REF** at (109.7, 71.8)
- removed the REF** at (183.2, 113.5)
- removed the REF** at (120.2, 71.8)
- removed the REF** at (120.4, 176.5)
- removed the REF** at (88.9, 155.4)
- removed the REF** at (120.2, 50.5)
- removed the REF** at (88.7, 50.4)
- removed the REF** at (25.7, 113.5)
- removed the REF** at (178.8, 82.5)
- removed the REF** at (88.7, 98.0)
- removed the REF** at (109.9, 155.5)
- removed the REF** at (57.1, 134.4)
- removed the REF** at (67.8, 113.5)
- removed the REF** at (120.2, 92.8)
- removed the REF** at (109.7, 92.8)
- removed the REF** at (46.7, 50.5)
- removed the REF** at (162.2, 134.5)
- removed the REF** at (36.2, 113.5)
- removed the REF** at (67.7, 56.0)
- removed the REF** at (25.9, 176.5)
- removed the REF** at (151.8, 113.5)
- removed the REF** at (67.8, 92.7)
- removed the REF** at (141.1, 134.5)
- removed the REF** at (116.0, 166.3)
- removed the REF** at (68.0, 155.5)
- removed the REF** at (173.0, 176.5)
- removed the REF** at (31.8, 124.2)
- removed the REF** at (95.0, 166.2)
- removed the REF** at (78.2, 56.0)
- removed the REF** at (88.7, 113.4)
- removed the REF** at (57.1, 113.5)
- removed the REF** at (162.5, 176.5)
- removed the REF** at (94.8, 82.5)
- removed the REF** at (36.2, 71.8)
- removed the REF** at (151.8, 71.8)
- removed the REF** at (99.2, 50.4)
- removed the REF** at (99.2, 71.7)
- removed the REF** at (109.7, 108.5)
- removed the REF** at (130.7, 50.5)
- removed the REF** at (57.4, 155.5)
- removed the REF** at (52.7, 82.5)
- removed the REF** at (141.4, 155.5)
- removed the REF** at (73.8, 124.2)
- removed the REF** at (78.5, 176.5)
- removed the REF** at (115.8, 124.3)
- removed the REF** at (189.0, 155.5)
- removed the REF** at (89.0, 176.4)
- removed the REF** at (109.7, 50.5)
- removed the REF** at (109.7, 134.5)
- removed the REF** at (78.5, 155.5)
- removed the REF** at (36.2, 50.5)
- removed the REF** at (183.2, 50.5)
- removed the REF** at (136.9, 166.3)
- removed the REF** at (158.1, 166.3)
- removed the REF** at (109.7, 119.0)
- removed the REF** at (162.2, 119.0)
- removed the REF** at (157.2, 113.5)
- removed the REF** at (31.0, 50.5)
- removed the REF** at (36.2, 24.5)
- removed the REF** at (52.2, 155.5)
- removed the REF** at (25.2, 166.2)
- removed the REF** at (25.7, 182.0)
- removed the REF** at (183.2, 45.5)
- removed the REF** at (141.2, 150.5)
- removed the REF** at (115.0, 71.8)
- removed the REF** at (73.2, 92.8)
- removed the REF** at (109.7, 77.0)
- removed the REF** at (126.0, 176.5)
- removed the REF** at (130.7, 45.5)
- removed the REF** at (84.0, 155.5)
- removed the REF** at (78.2, 108.5)
- removed the REF** at (172.2, 166.2)
- removed the REF** at (46.7, 119.0)
- removed the REF** at (183.2, 66.5)
- removed the REF** at (94.0, 92.8)
- removed the REF** at (136.0, 92.8)
- removed the REF** at (104.5, 50.5)
- removed the REF** at (25.7, 171.5)
- removed the REF** at (183.2, 161.0)
- removed the REF** at (57.2, 98.0)
- removed the REF** at (136.0, 50.5)
- removed the REF** at (31.0, 134.5)
- removed the REF** at (115.0, 134.5)
- removed the REF** at (67.7, 182.0)
- removed the REF** at (36.2, 98.0)
- removed the REF** at (46.7, 108.5)
- removed the REF** at (36.2, 45.5)
- removed the REF** at (31.2, 176.5)
- removed the REF** at (130.7, 171.5)
- removed the REF** at (99.2, 119.0)
- removed the REF** at (109.7, 150.5)
- removed the REF** at (99.2, 140.0)
Routing:
- net (no net): track 11415.2 -> 737.8 mm, vias 428 -> 78
Other:
- board outline removed
