File: hardware/KiCad/shematic1/shematic1.kicad_sch (KiCad schematic)
At the start: 1 part, among them u1 LFE5U-25F-6BG256C

Commit message: working cross-platform compilation
Parts:
- added U2: 74AHC1G00, symbol 74xGxx:74AHC1G00
Connections:
- net at u1.J1 (PL23A): now also u1.J2 (PL23B), u1.J3 (PL20C), U2.5 (VCC)
- net GND: now reaches u1.J10 (GND_16)
- net GND: now also u1.J8 (GND_14), u1.J9 (GND_15)
- net at u1.J12 (PR17D): now also U2.3 (GND)
- net at u1.J14 (PR20C): now also U2.4
- net at u1.J6 (VCCIO6_1): now also U2.1
- net at u1.J7 (VCCIO6_2): now also U2.2
Other:
- moved on the sheet: u1
