File: hardware/KiCad/shematic1/Transducer10.kicad_sch (KiCad schematic)
At the start: 14 parts, among them U52 74HC595D, U53 MIC4127YML-TR, U54 MIC4127YML-TR, U55 MIC4127YML-TR, U56 MIC4127YML-TR

Commit message: updated KiCad schematics
Parts:
- U207: renamed from U52; footprint SOIC16_TOS -> (none)
- U208: renamed from U53; footprint MLF-8_ML_MCH -> (none)
- U209: renamed from U54; footprint MLF-8_ML_MCH -> (none)
- U210: renamed from U55; footprint MLF-8_ML_MCH -> (none)
- U211: renamed from U56; footprint MLF-8_ML_MCH -> (none)
- renumbered C11 to C42, LS81 to LS329, LS82 to LS330, LS83 to LS331, LS84 to LS332, LS85 to LS333, LS86 to LS334, LS87 to LS335, LS88 to LS336
Connections:
- net +5V: now also U207.10 (*SCLR)
- net GND: now also U207.13 (*G), U207.8 (GND), U208.3 (GND), U209.3 (GND), U210.3 (GND), U211.3 (GND)
- net SCK: now reaches U207.11 (SCK)
- net RCK: now reaches U207.12 (RCK)
- net In renamed SI_T10
- no-connect marks 0 -> 5
Other:
- note removed: "GND"

Commit message: modified pcb
Parts:
- removed C42: 0.1μF, symbol Device:C_Small
- added C19, C20: 0.1μF, symbol Device:C_Small
Connections:
- net VCC is gone; now on net +5V: U208.6 (VS), U209.6 (VS), U210.6 (VS), U211.6 (VS)
- net +5V: now also C20.1; no longer U207.10 (*SCLR), U207.16 (VCC)
- net GND: now also C19.2, C20.2
- new net +3.3V: C19.1, U207.10 (*SCLR), U207.16 (VCC)
