File: hardware/KiCad/shematic1/Transducer11.kicad_sch (KiCad schematic)
At the start: 14 parts, among them U57 74HC595D, U58 MIC4127YML-TR, U59 MIC4127YML-TR, U60 MIC4127YML-TR, U61 MIC4127YML-TR

Commit message: updated KiCad schematics
Parts:
- U212: renamed from U57; footprint SOIC16_TOS -> (none)
- U213: renamed from U58; footprint MLF-8_ML_MCH -> (none)
- U214: renamed from U59; footprint MLF-8_ML_MCH -> (none)
- U215: renamed from U60; footprint MLF-8_ML_MCH -> (none)
- U216: renamed from U61; footprint MLF-8_ML_MCH -> (none)
- renumbered C12 to C43, LS89 to LS337, LS90 to LS338, LS91 to LS339, LS92 to LS340, LS93 to LS341, LS94 to LS342, LS95 to LS343, LS96 to LS344
Connections:
- net +5V: now also U212.10 (*SCLR)
- net GND: now also U212.13 (*G), U212.8 (GND), U213.3 (GND), U214.3 (GND), U215.3 (GND), U216.3 (GND)
- net SCK: now reaches U212.11 (SCK)
- net RCK: now reaches U212.12 (RCK)
- net In renamed SI_T11
- no-connect marks 0 -> 5
Other:
- note removed: "GND"

Commit message: modified pcb
Parts:
- removed C43: 0.1μF, symbol Device:C_Small
- added C21, C22: 0.1μF, symbol Device:C_Small
Connections:
- net VCC is gone; now on net +5V: U213.6 (VS), U214.6 (VS), U215.6 (VS), U216.6 (VS)
- net +5V: now also C22.1; no longer U212.10 (*SCLR), U212.16 (VCC)
- net GND: now also C21.2, C22.2
- new net +3.3V: C21.1, U212.10 (*SCLR), U212.16 (VCC)
