File: hardware/KiCad/shematic1/Transducer12.kicad_sch (KiCad schematic)
At the start: 14 parts, among them U62 74HC595D, U63 MIC4127YML-TR, U64 MIC4127YML-TR, U65 MIC4127YML-TR, U66 MIC4127YML-TR

Commit message: updated KiCad schematics
Parts:
- U217: renamed from U62; footprint SOIC16_TOS -> (none)
- U218: renamed from U63; footprint MLF-8_ML_MCH -> (none)
- U219: renamed from U64; footprint MLF-8_ML_MCH -> (none)
- U220: renamed from U65; footprint MLF-8_ML_MCH -> (none)
- U221: renamed from U66; footprint MLF-8_ML_MCH -> (none)
- renumbered C13 to C44, LS97 to LS345, LS98 to LS346, LS99 to LS347, LS100 to LS348, LS101 to LS349, LS102 to LS350, LS103 to LS351, LS104 to LS352
Connections:
- net +5V: now also U217.10 (*SCLR)
- net GND: now also U217.13 (*G), U217.8 (GND), U218.3 (GND), U219.3 (GND), U220.3 (GND), U221.3 (GND)
- net SCK: now reaches U217.11 (SCK)
- net RCK: now reaches U217.12 (RCK)
- net In renamed SI_T12
- no-connect marks 0 -> 5
Other:
- note removed: "GND"

Commit message: modified pcb
Parts:
- removed C44: 0.1μF, symbol Device:C_Small
- added C23, C24: 0.1μF, symbol Device:C_Small
Connections:
- net VCC is gone; now on net +5V: U218.6 (VS), U219.6 (VS), U220.6 (VS), U221.6 (VS)
- net +5V: now also C24.1; no longer U217.10 (*SCLR), U217.16 (VCC)
- net GND: now also C23.2, C24.2
- new net +3.3V: C23.1, U217.10 (*SCLR), U217.16 (VCC)
