File: hardware/KiCad/shematic1/Transducer14.kicad_sch (KiCad schematic)
At the start: 14 parts, among them U72 74HC595D, U73 MIC4127YML-TR, U74 MIC4127YML-TR, U75 MIC4127YML-TR, U76 MIC4127YML-TR

Commit message: updated KiCad schematics
Parts:
- U227: renamed from U72; footprint SOIC16_TOS -> (none)
- U228: renamed from U73; footprint MLF-8_ML_MCH -> (none)
- U229: renamed from U74; footprint MLF-8_ML_MCH -> (none)
- U230: renamed from U75; footprint MLF-8_ML_MCH -> (none)
- U231: renamed from U76; footprint MLF-8_ML_MCH -> (none)
- renumbered C15 to C46, LS113 to LS361, LS114 to LS362, LS115 to LS363, LS116 to LS364, LS117 to LS365, LS118 to LS366, LS119 to LS367, LS120 to LS368
Connections:
- net +5V: now also U227.10 (*SCLR)
- net GND: now also U227.13 (*G), U227.8 (GND), U228.3 (GND), U229.3 (GND), U230.3 (GND), U231.3 (GND)
- net SCK: now reaches U227.11 (SCK)
- net RCK: now reaches U227.12 (RCK)
- net In renamed SI_T14
- no-connect marks 0 -> 5
Other:
- note removed: "GND"

Commit message: modified pcb
Parts:
- removed C46: 0.1μF, symbol Device:C_Small
- added C27, C28: 0.1μF, symbol Device:C_Small
Connections:
- net VCC is gone; now on net +5V: U228.6 (VS), U229.6 (VS), U230.6 (VS), U231.6 (VS)
- net +5V: now also C28.1; no longer U227.10 (*SCLR), U227.16 (VCC)
- net GND: now also C27.2, C28.2
- new net +3.3V: C27.1, U227.10 (*SCLR), U227.16 (VCC)
