File: hardware/KiCad/shematic1/Transducer15.kicad_sch (KiCad schematic)
At the start: 14 parts, among them U77 74HC595D, U78 MIC4127YML-TR, U79 MIC4127YML-TR, U80 MIC4127YML-TR, U81 MIC4127YML-TR

Commit message: updated KiCad schematics
Parts:
- U232: renamed from U77; footprint SOIC16_TOS -> (none)
- U233: renamed from U78; footprint MLF-8_ML_MCH -> (none)
- U234: renamed from U79; footprint MLF-8_ML_MCH -> (none)
- U235: renamed from U80; footprint MLF-8_ML_MCH -> (none)
- U236: renamed from U81; footprint MLF-8_ML_MCH -> (none)
- renumbered C16 to C47, LS121 to LS369, LS122 to LS370, LS123 to LS371, LS124 to LS372, LS125 to LS373, LS126 to LS374, LS127 to LS375, LS128 to LS376
Connections:
- net +5V: now also U232.10 (*SCLR)
- net GND: now also U232.13 (*G), U232.8 (GND), U233.3 (GND), U234.3 (GND), U235.3 (GND), U236.3 (GND)
- net SCK: now reaches U232.11 (SCK)
- net RCK: now reaches U232.12 (RCK)
- net In renamed SI_T15
- no-connect marks 0 -> 5
Other:
- note removed: "GND"

Commit message: modified pcb
Parts:
- removed C47: 0.1μF, symbol Device:C_Small
- added C29, C30: 0.1μF, symbol Device:C_Small
Connections:
- net VCC is gone; now on net +5V: U233.6 (VS), U234.6 (VS), U235.6 (VS), U236.6 (VS)
- net +5V: now also C30.1; no longer U232.10 (*SCLR), U232.16 (VCC)
- net GND: now also C29.2, C30.2
- new net +3.3V: C29.1, U232.10 (*SCLR), U232.16 (VCC)
