File: hardware/KiCad/shematic1/Transducer17.kicad_sch (KiCad schematic)
At the start: 14 parts, among them U87 74HC595D, U88 MIC4127YML-TR, U89 MIC4127YML-TR, U90 MIC4127YML-TR, U91 MIC4127YML-TR

Commit message: updated KiCad schematics
Parts:
- U242: renamed from U87; footprint SOIC16_TOS -> (none)
- U243: renamed from U88; footprint MLF-8_ML_MCH -> (none)
- U244: renamed from U89; footprint MLF-8_ML_MCH -> (none)
- U245: renamed from U90; footprint MLF-8_ML_MCH -> (none)
- U246: renamed from U91; footprint MLF-8_ML_MCH -> (none)
- renumbered C18 to C49, LS137 to LS385, LS138 to LS386, LS139 to LS387, LS140 to LS388, LS141 to LS389, LS142 to LS390, LS143 to LS391, LS144 to LS392
Connections:
- net +5V: now also U242.10 (*SCLR)
- net GND: now also U242.13 (*G), U242.8 (GND), U243.3 (GND), U244.3 (GND), U245.3 (GND)
- net SCK: now reaches U242.11 (SCK)
- net RCK: now reaches U242.12 (RCK)
- net In renamed SI_T17
- no-connect marks 0 -> 5
Other:
- note removed: "GND"

Commit message: modified pcb
Parts:
- removed C49: 0.1μF, symbol Device:C_Small
- added C33, C34: 0.1μF, symbol Device:C_Small
Connections:
- net VCC is gone; now on net +5V: U243.6 (VS), U244.6 (VS), U245.6 (VS), U246.6 (VS)
- net +5V: now also C34.1; no longer U242.10 (*SCLR), U242.16 (VCC)
- net GND: now also C33.2, C34.2
- new net +3.3V: C33.1, U242.10 (*SCLR), U242.16 (VCC)
