File: hardware/KiCad/shematic1/Transducer2.kicad_sch (KiCad schematic)
At the start: 14 parts, among them U12 74HC595D, U13 MIC4127YML-TR, U14 MIC4127YML-TR, U15 MIC4127YML-TR, U16 MIC4127YML-TR

Commit message: updated KiCad schematics
Parts:
- U167: renamed from U12; footprint SOIC16_TOS -> (none)
- U168: renamed from U13; footprint MLF-8_ML_MCH -> (none)
- U169: renamed from U14; footprint MLF-8_ML_MCH -> (none)
- U170: renamed from U15; footprint MLF-8_ML_MCH -> (none)
- U171: renamed from U16; footprint MLF-8_ML_MCH -> (none)
- renumbered C3 to C34, LS17 to LS265, LS18 to LS266, LS19 to LS267, LS20 to LS268, LS21 to LS269, LS22 to LS270, LS23 to LS271, LS24 to LS272
Connections:
- net +5V: now also U167.10 (*SCLR)
- net GND: now also U167.13 (*G), U167.8 (GND), U168.3 (GND), U169.3 (GND), U170.3 (GND), U171.3 (GND)
- net SCK: now reaches U167.11 (SCK)
- net RCK: now reaches U167.12 (RCK)
- net In renamed SI_T2
- no-connect marks 0 -> 5
Other:
- note removed: "GND"

Commit message: modified pcb
Parts:
- removed C34: 0.1μF, symbol Device:C_Small
- added C3, C4: 0.1μF, symbol Device:C_Small
Connections:
- net VCC is gone; now on net +5V: U168.6 (VS), U169.6 (VS), U170.6 (VS), U171.6 (VS)
- net +5V: now also C4.1; no longer U167.10 (*SCLR), U167.16 (VCC)
- net GND: now also C3.2, C4.2
- new net +3.3V: C3.1, U167.10 (*SCLR), U167.16 (VCC)
