File: hardware/KiCad/shematic1/Transducer24.kicad_sch (KiCad schematic)
At the start: 14 parts, among them U122 74HC595D, U123 MIC4127YML-TR, U124 MIC4127YML-TR, U125 MIC4127YML-TR, U126 MIC4127YML-TR

Commit message: updated KiCad schematics
Parts:
- U277: renamed from U122; footprint SOIC16_TOS -> (none)
- U278: renamed from U123; footprint MLF-8_ML_MCH -> (none)
- U279: renamed from U124; footprint MLF-8_ML_MCH -> (none)
- U280: renamed from U125; footprint MLF-8_ML_MCH -> (none)
- U281: renamed from U126; footprint MLF-8_ML_MCH -> (none)
- renumbered C25 to C56, LS193 to LS441, LS194 to LS442, LS195 to LS443, LS196 to LS444, LS197 to LS445, LS198 to LS446, LS199 to LS447, LS200 to LS448
Connections:
- net +5V: now also U277.10 (*SCLR)
- net GND: now also U277.13 (*G), U277.8 (GND), U278.3 (GND), U279.3 (GND), U280.3 (GND), U281.3 (GND)
- net SCK: now reaches U277.11 (SCK)
- net RCK: now reaches U277.12 (RCK)
- net In renamed SI_T24
- no-connect marks 0 -> 5
Other:
- note removed: "GND"

Commit message: modified pcb
Parts:
- removed C56: 0.1μF, symbol Device:C_Small
- added C47, C48: 0.1μF, symbol Device:C_Small
Connections:
- net VCC is gone; now on net +5V: U278.6 (VS), U279.6 (VS), U280.6 (VS), U281.6 (VS)
- net +5V: now also C48.1; no longer U277.10 (*SCLR), U277.16 (VCC)
- net GND: now also C47.2, C48.2
- new net +3.3V: C47.1, U277.10 (*SCLR), U277.16 (VCC)
