File: hardware/KiCad/shematic1/Transducer25.kicad_sch (KiCad schematic)
At the start: 14 parts, among them U127 74HC595D, U128 MIC4127YML-TR, U129 MIC4127YML-TR, U130 MIC4127YML-TR, U131 MIC4127YML-TR

Commit message: updated KiCad schematics
Parts:
- U282: renamed from U127; footprint SOIC16_TOS -> (none)
- U283: renamed from U128; footprint MLF-8_ML_MCH -> (none)
- U284: renamed from U129; footprint MLF-8_ML_MCH -> (none)
- U285: renamed from U130; footprint MLF-8_ML_MCH -> (none)
- U286: renamed from U131; footprint MLF-8_ML_MCH -> (none)
- renumbered C26 to C57, LS201 to LS449, LS202 to LS450, LS203 to LS451, LS204 to LS452, LS205 to LS453, LS206 to LS454, LS207 to LS455, LS208 to LS456
Connections:
- net +5V: now also U282.10 (*SCLR)
- net GND: now also U282.13 (*G), U282.8 (GND), U283.3 (GND), U284.3 (GND), U285.3 (GND), U286.3 (GND)
- net SCK: now reaches U282.11 (SCK)
- net RCK: now reaches U282.12 (RCK)
- net In renamed SI_T25
- no-connect marks 0 -> 5
Other:
- note removed: "GND"

Commit message: modified pcb
Parts:
- removed C57: 0.1μF, symbol Device:C_Small
- added C49, C50: 0.1μF, symbol Device:C_Small
Connections:
- net VCC is gone; now on net +5V: U283.6 (VS), U284.6 (VS), U285.6 (VS), U286.6 (VS)
- net +5V: now also C50.1; no longer U282.10 (*SCLR), U282.16 (VCC)
- net GND: now also C49.2, C50.2
- new net +3.3V: C49.1, U282.10 (*SCLR), U282.16 (VCC)
