File: hardware/KiCad/shematic1/Transducer28.kicad_sch (KiCad schematic)
At the start: 14 parts, among them U142 74HC595D, U143 MIC4127YML-TR, U144 MIC4127YML-TR, U145 MIC4127YML-TR, U146 MIC4127YML-TR

Commit message: updated KiCad schematics
Parts:
- U297: renamed from U142; footprint SOIC16_TOS -> (none)
- U298: renamed from U143; footprint MLF-8_ML_MCH -> (none)
- U299: renamed from U144; footprint MLF-8_ML_MCH -> (none)
- U300: renamed from U145; footprint MLF-8_ML_MCH -> (none)
- U301: renamed from U146; footprint MLF-8_ML_MCH -> (none)
- renumbered C29 to C60, LS225 to LS473, LS226 to LS474, LS227 to LS475, LS228 to LS476, LS229 to LS477, LS230 to LS478, LS231 to LS479, LS232 to LS480
Connections:
- net +5V: now also U297.10 (*SCLR)
- net GND: now also U297.13 (*G), U297.8 (GND), U298.3 (GND), U299.3 (GND), U300.3 (GND), U301.3 (GND)
- net SCK: now reaches U297.11 (SCK)
- net RCK: now reaches U297.12 (RCK)
- net In renamed SI_T28
- no-connect marks 0 -> 5
Other:
- note removed: "GND"

Commit message: modified pcb
Parts:
- removed C60: 0.1μF, symbol Device:C_Small
- added C55, C56: 0.1μF, symbol Device:C_Small
Connections:
- net VCC is gone; now on net +5V: U298.6 (VS), U299.6 (VS), U300.6 (VS), U301.6 (VS)
- net +5V: now also C56.1; no longer U297.10 (*SCLR), U297.16 (VCC)
- net GND: now also C55.2, C56.2
- new net +3.3V: C55.1, U297.10 (*SCLR), U297.16 (VCC)
