File: hardware/KiCad/shematic1/Transducer29.kicad_sch (KiCad schematic)
At the start: 14 parts, among them U147 74HC595D, U148 MIC4127YML-TR, U149 MIC4127YML-TR, U150 MIC4127YML-TR, U151 MIC4127YML-TR

Commit message: updated KiCad schematics
Parts:
- U302: renamed from U147; footprint SOIC16_TOS -> (none)
- U303: renamed from U148; footprint MLF-8_ML_MCH -> (none)
- U304: renamed from U149; footprint MLF-8_ML_MCH -> (none)
- U305: renamed from U150; footprint MLF-8_ML_MCH -> (none)
- U306: renamed from U151; footprint MLF-8_ML_MCH -> (none)
- renumbered C30 to C61, LS233 to LS481, LS234 to LS482, LS235 to LS483, LS236 to LS484, LS237 to LS485, LS238 to LS486, LS239 to LS487, LS240 to LS488
Connections:
- net +5V: now also U302.10 (*SCLR)
- net GND: now also U302.13 (*G), U302.8 (GND), U303.3 (GND), U304.3 (GND), U305.3 (GND), U306.3 (GND)
- net SCK: now reaches U302.11 (SCK)
- net RCK: now reaches U302.12 (RCK)
- net In renamed SI_T29
- no-connect marks 0 -> 5
Other:
- note removed: "GND"

Commit message: modified pcb
Parts:
- removed C61: 0.1μF, symbol Device:C_Small
- added C57, C58: 0.1μF, symbol Device:C_Small
Connections:
- net VCC is gone; now on net +5V: U303.6 (VS), U304.6 (VS), U305.6 (VS), U306.6 (VS)
- net +5V: now also C58.1; no longer U302.10 (*SCLR), U302.16 (VCC)
- net GND: now also C57.2, C58.2
- new net +3.3V: C57.1, U302.10 (*SCLR), U302.16 (VCC)
