File: hardware/KiCad/shematic1/Transducer3.kicad_sch (KiCad schematic)
At the start: 14 parts, among them U17 74HC595D, U18 MIC4127YML-TR, U19 MIC4127YML-TR, U20 MIC4127YML-TR, U21 MIC4127YML-TR

Commit message: updated KiCad schematics
Parts:
- U172: renamed from U17; footprint SOIC16_TOS -> (none)
- U173: renamed from U18; footprint MLF-8_ML_MCH -> (none)
- U174: renamed from U19; footprint MLF-8_ML_MCH -> (none)
- U175: renamed from U20; footprint MLF-8_ML_MCH -> (none)
- U176: renamed from U21; footprint MLF-8_ML_MCH -> (none)
- renumbered C4 to C35, LS25 to LS273, LS26 to LS274, LS27 to LS275, LS28 to LS276, LS29 to LS277, LS30 to LS278, LS31 to LS279, LS32 to LS280
Connections:
- net +5V: now also U172.10 (*SCLR)
- net GND: now also U172.13 (*G), U172.8 (GND), U173.3 (GND), U174.3 (GND), U175.3 (GND), U176.3 (GND)
- net SCK: now reaches U172.11 (SCK)
- net RCK: now reaches U172.12 (RCK)
- net In renamed SI_T3
- no-connect marks 0 -> 5
Other:
- note removed: "GND"

Commit message: modified pcb
Parts:
- removed C35: 0.1μF, symbol Device:C_Small
- added C5, C6: 0.1μF, symbol Device:C_Small
Connections:
- net VCC is gone; now on net +5V: U173.6 (VS), U174.6 (VS), U175.6 (VS), U176.6 (VS)
- net +5V: now also C6.1; no longer U172.10 (*SCLR), U172.16 (VCC)
- net GND: now also C5.2, C6.2
- new net +3.3V: C5.1, U172.10 (*SCLR), U172.16 (VCC)
