File: hardware/KiCad/shematic1/Transducer30.kicad_sch (KiCad schematic)
At the start: 14 parts, among them U152 74HC595D, U153 MIC4127YML-TR, U154 MIC4127YML-TR, U155 MIC4127YML-TR, U156 MIC4127YML-TR

Commit message: updated KiCad schematics
Parts:
- U307: renamed from U152; footprint SOIC16_TOS -> (none)
- U308: renamed from U153; footprint MLF-8_ML_MCH -> (none)
- U309: renamed from U154; footprint MLF-8_ML_MCH -> (none)
- U310: renamed from U155; footprint MLF-8_ML_MCH -> (none)
- U311: renamed from U156; footprint MLF-8_ML_MCH -> (none)
- renumbered C31 to C62, LS241 to LS489, LS242 to LS490, LS243 to LS491, LS244 to LS492, LS245 to LS493, LS246 to LS494, LS247 to LS495, LS248 to LS496
Connections:
- net +5V: now also U307.10 (*SCLR)
- net GND: now also U307.13 (*G), U307.8 (GND), U308.3 (GND), U309.3 (GND), U310.3 (GND), U311.3 (GND)
- net SCK: now reaches U307.11 (SCK)
- net RCK: now reaches U307.12 (RCK)
- net In renamed SI_T30
- no-connect marks 0 -> 5
Other:
- note removed: "GND"

Commit message: modified pcb
Parts:
- removed C62: 0.1μF, symbol Device:C_Small
- added C59, C60: 0.1μF, symbol Device:C_Small
Connections:
- net VCC is gone; now on net +5V: U308.6 (VS), U309.6 (VS), U310.6 (VS), U311.6 (VS)
- net +5V: now also C60.1; no longer U307.10 (*SCLR), U307.16 (VCC)
- net GND: now also C59.2, C60.2
- new net +3.3V: C59.1, U307.10 (*SCLR), U307.16 (VCC)
