File: hardware/KiCad/shematic1/Transducer7.kicad_sch (KiCad schematic)
At the start: 14 parts, among them U37 74HC595D, U38 MIC4127YML-TR, U39 MIC4127YML-TR, U40 MIC4127YML-TR, U41 MIC4127YML-TR

Commit message: updated KiCad schematics
Parts:
- U192: renamed from U37; footprint SOIC16_TOS -> (none)
- U193: renamed from U38; footprint MLF-8_ML_MCH -> (none)
- U194: renamed from U39; footprint MLF-8_ML_MCH -> (none)
- U195: renamed from U40; footprint MLF-8_ML_MCH -> (none)
- U196: renamed from U41; footprint MLF-8_ML_MCH -> (none)
- renumbered C8 to C39, LS57 to LS305, LS58 to LS306, LS59 to LS307, LS60 to LS308, LS61 to LS309, LS62 to LS310, LS63 to LS311, LS64 to LS312
Connections:
- net +5V: now also U192.10 (*SCLR)
- net GND: now also U192.13 (*G), U192.8 (GND), U193.3 (GND), U194.3 (GND), U195.3 (GND), U196.3 (GND)
- net SCK: now reaches U192.11 (SCK)
- net RCK: now reaches U192.12 (RCK)
- net In renamed SI_T7
- no-connect marks 0 -> 5
Other:
- note removed: "GND"

Commit message: modified pcb
Parts:
- removed C39: 0.1μF, symbol Device:C_Small
- added C13, C14: 0.1μF, symbol Device:C_Small
Connections:
- net VCC is gone; now on net +5V: U193.6 (VS), U194.6 (VS), U195.6 (VS), U196.6 (VS)
- net +5V: now also C14.1; no longer U192.10 (*SCLR), U192.16 (VCC)
- net GND: now also C13.2, C14.2
- new net +3.3V: C13.1, U192.10 (*SCLR), U192.16 (VCC)
