File: hardware/fpgapcb/.history/link.kicad_sch (KiCad schematic)
At the start: 68 parts, among them J1 Conn_01x03_Pin, J2 JTAG, J4 Screw_Terminal_01x02, U10 TLV62569DBV, U7 W25Q32JVSS, U8 TPS54302, U9 TLV62569DBV, u2 LFE5U-25F-6BG256C

Commit message: add new schem
Parts:
- removed u2: LFE5U-25F-6BG256C, Package_BGA:LFBGA-289_14x14mm_Layout17x17_P0.8mm, symbol FPGA_LFE5U-25F-6BG256C:LFE5U-25F-6BG256C
- added U5: (no value), symbol LFE5U-25F-6TG144C:LFE5U-25F-6TG144C
Connections:
- net CSS: now also U5.91 (PR23A)
- net DONE: now also U5.56 (DONE)
- net GND: now also U5.101 (GND), U5.123 (GND), U5.129 (GND), U5.131 (GND), U5.138 (GND), U5.15 (GND), U5.21 (GND), U5.42 (GND), U5.65 (GND), U5.75 (GND), U5.8 (GND), U5.85 (GND), U5.87 (GND)
- net IO2: now also U5.77 (PR41A)
- net IO3: now also U5.74 (PR41C)
- net MCLK: now also U5.54 (CCLK)
- net MISO/D1: now also U5.89 (PR23B)
- net MOSI/D0: now also U5.90 (PR23C)
- net PROGRAMN: now also U5.57 (PROGRAMN)
- net RCK: now also U5.44 (PB4B)
- net SCK: now also U5.41 (PB6B)
- net SI_T1: now also U5.1 (PL5C)
- net SI_T10: now also U5.11 (PL14C)
- net SI_T11: now also U5.12 (PL14B)
- net SI_T12: now also U5.13 (PL14D)
- net SI_T13: now also U5.14 (PL23D)
- net SI_T14: now also U5.18 (PL32B)
- net SI_T15: now also U5.26 (PL41C)
- net SI_T16: now also U5.27 (PL41D)
- net SI_T17: now also U5.31 (PL44C)
- net SI_T18: now also U5.30 (PL44B)
- net SI_T19: now also U5.33 (PL44D)
- net SI_T2: now also U5.2 (PL5D)
- net SI_T20: now also U5.35 (PL47B)
- net SI_T21: now also U5.46 (PB11A)
- net SI_T22: now also U5.45 (PB9A)
- net SI_T23: now also U5.37 (PL47C)
- net SI_T24: now also U5.47 (PB11B)
- net SI_T25: now also U5.49 (PB15A)
- net SI_T26: now also U5.50 (PB13B)
- net SI_T27: now also U5.51 (PB15B)
- net SI_T28: now also U5.52 (PL18A)
- net SI_T29: now also U5.71 (PR47A)
- net SI_T3: now also U5.3 (PL5B)
- net SI_T30: now also U5.72 (PR44C)
- net SI_T31: now also U5.73 (PR41D)
- net SI_T32: now also U5.76 (PR41B)
- net SI_T4: now also U5.4 (PL8A)
- net SI_T5: now also U5.5 (PL8C)
- net SI_T6: now also U5.24 (PL38A)
- net SI_T7: now also U5.25 (PL38B)
- net SI_T8: now also U5.6 (PL8B)
- net SI_T9: now also U5.10 (PL14A)
- net TCK: now also U5.63 (TCK)
- net TDI: now also U5.61 (TDI)
- net TDO: now also U5.60 (TDO)
- net TMS: now also U5.64 (TMS)
- new net INITN: U5.55 (INITN)
- no-connect marks 161 -> 5
Other:
- moved on the sheet: C100, C101, C102, C103, C104, C105, C106, C107, C108, C65, C66, C67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

Commit message: madameng kabadengan ang nangyare - finished connections & putprint
Connections:
- net +1V1: now also U5.130 (VCC), U5.20 (VCC), U5.29 (VCC), U5.38 (VCC), U5.66 (VCC), U5.83 (VCC)
- net +2V5: now also U5.132 (VCCAUX), U5.17 (VCCAUX), U5.53 (VCCAUX), U5.96 (VCCAUX)
- net +3.3V: now also R1.1, R3.1, U5.100 (VCCIO2), U5.122 (VCCIO1), U5.137 (VCCIO0), U5.16 (VCCIO6), U5.32 (VSSIO6), U5.36 (VCCIO6), U5.43 (VCIO8), U5.70 (VCCIO3), U5.86 (VCCIO3), U5.9 (VCCIO7)
- net GND: now also R2.2, U5.58 (CFG_2), U5.59 (CFG_1), U5.62 (CFG_0)
Other:
- moved on the sheet: J1, J2, R10, R11, R12, R13, R4, R5, R6, R7, R8, R9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

Commit message: add pins
Parts:
- added J3, J5: Conn_02x13_Odd_Even_MountingPin, symbol Connector_Generic_MountingPin:Conn_02x13_Odd_Even_MountingPin
- added J6, J7: Conn_02x13_Odd_Even, symbol Connector_Generic:Conn_02x13_Odd_Even
- added J8: Conn_02x05_Odd_Even, symbol Connector_Generic:Conn_02x05_Odd_Even

Commit message: added pins and connections
Parts:
- removed J1: Conn_01x03_Pin, Connector:FanPinHeader_1x03_P2.54mm_Vertical, symbol Connector:Conn_01x03_Pin
- removed J3, J5: Conn_02x13_Odd_Even_MountingPin, symbol Connector_Generic_MountingPin:Conn_02x13_Odd_Even_MountingPin
- added D3, D4, D5, D6, D7, D8: LED, symbol Device:LED
- added R20, R21, R22: 600, symbol Device:R_Small_US
- added U166, U2: CH340C, Package_SO:SOIC-16_3.9x9.9mm_P1.27mm, symbol Interface_USB:CH340C
- J6: value Conn_02x13_Odd_Even -> Channel A
- J7: value Conn_02x13_Odd_Even -> Channel B
Connections:
- net +1V1: now also D6.2 (A)
- net +2V5: now also D8.2 (A)
- net +3.3V: now also D7.2 (A); no longer R1.1, R3.1
- net DONE: now also D3.2 (A)
- net GND: now also D6.1 (K), D7.1 (K), D8.1 (K), R20.2, R21.2, R22.2; no longer R2.2, U5.58 (CFG_2), U5.59 (CFG_1), U5.62 (CFG_0)
- net INITN: now also D4.2 (A)
- net PROGRAMN: now also D5.2 (A)
- net TCK: now also J7.4 (Pin_4)
- net TDI: now also J7.6 (Pin_6)
- net TDO: now also J7.2 (Pin_2)
- net TMS: now also J7.8 (Pin_8)
- net io1: now reaches J6.1 (Pin_1)
- net io1: now also U5.121 (PT51A)
- net io6: now reaches J6.11 (Pin_11)
- net io6: now also U5.117 (PT56B)
- net io7: now reaches J6.13 (Pin_13)
- net io7: now also U5.115 (PT58B)
- net io8: now reaches J6.15 (Pin_15)
- net io8: now also U5.114 (PT60A)
- net io2: now reaches J6.3 (Pin_3)
- net io2: now also U5.120 (PT53A)
- net io3: now reaches J6.5 (Pin_5)
- net io3: now also U5.119 (PT53B)
- net io4: now reaches J6.7 (Pin_7)
- net io4: now also U5.118 (PT56A)
- net io5: now reaches J6.9 (Pin_9)
- net io5: now also U5.116 (PT58A)
- new net: D5.1 (K), R20.1
- new net: D4.1 (K), R21.1
- new net: D3.1 (K), R22.1
- new net CFG_0: R3.1, U5.62 (CFG_0)
- new net CFG_1: R2.2, U5.59 (CFG_1)
- new net CFG_2: R1.1, U5.58 (CFG_2)
- no-connect marks 5 -> 4
Other:
- moved on the sheet: J6, J7, J8, R1, R2, R3

Commit message: added more connections
Parts:
- removed U166: CH340C, Package_SO:SOIC-16_3.9x9.9mm_P1.27mm, symbol Interface_USB:CH340C
- added J1: Conn_01x06, symbol Connector_Generic:Conn_01x06
Connections:
- net +3.3V: now also J6.1 (Pin_1), J6.11 (Pin_11), J6.21 (Pin_21), J6.3 (Pin_3), J6.5 (Pin_5), J7.12 (Pin_12), J7.22 (Pin_22)
- net CSS: now also U5.80 (PR35C); no longer U5.91 (PR23A)
- net GND: now also J6.2 (Pin_2), J6.4 (Pin_4), J6.6 (Pin_6), J7.2 (Pin_2), J7.4 (Pin_4), U2.1 (GND), J1.1 (Pin_1)
- net MISO/D1: now also U5.78 (PR35D); no longer U5.89 (PR23B)
- net MOSI/D0: now also U5.79 (PR35B); no longer U5.90 (PR23C)
- net TCK: now also J7.26 (Pin_26); no longer J7.4 (Pin_4)
- net TDI: now also J7.25 (Pin_25); no longer J7.6 (Pin_6)
- net TDO: now also J7.24 (Pin_24); no longer J7.2 (Pin_2)
- net TMS: now also J7.23 (Pin_23); no longer J7.8 (Pin_8)
- net D1: now reaches J6.10 (Pin_10)
- net D1: now also U5.120 (PT53A)
- net D3: now reaches J6.12 (Pin_12)
- net D3: now also U5.118 (PT56A)
- net D4: now reaches J6.14 (Pin_14)
- net D4: now also U5.116 (PT58A)
- net D6: now reaches J6.16 (Pin_16)
- net D6: now also U5.115 (PT58B)
- net TXE#: now reaches J6.17 (Pin_17)
- net TXE#: now also U5.134 (PT15A)
- net RXF#: now reaches J6.18 (Pin_18)
- net RXF#: now also U5.136 (PT13A)
- net WR#: now reaches J6.19 (Pin_19)
- net WR#: now also U5.133 (PT15B)
- net RD#: now reaches J6.20 (Pin_20)
- net RD#: now also U5.135 (PT13B)
- net OE#: now reaches J6.23 (Pin_23)
- net OE#: now also U5.128 (PT29A)
- net CLKOUT: now reaches J6.24 (Pin_24)
- net CLKOUT: now also U5.88 (PR23D)
- net TXO: now reaches U2.2 (TXD)
- net TXO: now also U5.112 (PT62A), J1.2 (Pin_2)
- net RXI: now reaches U2.3 (RXD)
- net RXI: now also U5.113 (PT60B), J1.3 (Pin_3)
- net +5V: now reaches J7.5 (Pin_5)
- net io1 renamed D0
- net D0: now also J6.7 (Pin_7); no longer J6.1 (Pin_1)
- removed net io2: J6.3 (Pin_3), U5.120 (PT53A)
- net io3 renamed D2
- net D2: now also J6.9 (Pin_9); no longer J6.5 (Pin_5)
- removed net io4: J6.7 (Pin_7), U5.118 (PT56A)
- removed net io5: J6.9 (Pin_9), U5.116 (PT58A)
- net io6 renamed D5
- net D5: now also J6.13 (Pin_13); no longer J6.11 (Pin_11)
- removed net io7: J6.13 (Pin_13), U5.115 (PT58B)
- net io8 renamed D7

Commit message: reconstruct connections
Parts:
- removed J2: JTAG, Connector_IDC:IDC-Header_2x05_P2.54mm_Vertical, symbol Connector_Generic:Conn_02x05_Odd_Even
- removed R4, R5, R6, R7: 4.7K, Resistor_SMD:R_0805_2012Metric, symbol Device:R_Small_US
- removed U5: (no value), symbol LFE5U-25F-6TG144C:LFE5U-25F-6TG144C
- added D10, D11, D12, D9: LED, symbol Device:LED
- added R23, R24, R25, R26: 600, symbol Device:R_Small_US
- added R27, R28, R29, R30: 4.7K, Resistor_SMD:R_0805_2012Metric, symbol Device:R_Small_US
- added SW1: SW_MEC_5G_LED, symbol Switch:SW_MEC_5G_LED
- added U166: (no value), symbol LFE5U-25F-7TG144C:LFE5U-25F-7TG144C
Connections:
- net +1V1: now also U166.130 (VCC), U166.20 (VCC), U166.29 (VCC), U166.38 (VCC), U166.66 (VCC), U166.83 (VCC)
- net +2V5: now also U166.132 (VCCAUX), U166.17 (VCCAUX), U166.53 (VCCAUX), U166.96 (VCCAUX)
- net +3.3V: now also R27.2, R28.2, R30.1, U166.100 (VCCIO2), U166.122 (VCCIO1), U166.137 (VCCIO0), U166.16 (VCCIO6), U166.32 (VSSIO6), U166.36 (VCCIO6), U166.43 (VCIO8), U166.70 (VCCIO3), U166.86 (VCCIO3), U166.9 (VCCIO7)
- net +5V: now also J7.1 (Pin_1), J7.3 (Pin_3); no longer J7.5 (Pin_5)
- net CFG_0: now also U166.62 (CFG_0)
- net CFG_1: now also U166.59 (CFG_1)
- net CFG_2: now also U166.58 (CFG_2)
- net CLKOUT: now also U166.88 (PR23D)
- net CSS: now also U166.80 (PR35C)
- net D0: now also U166.121 (PT51A)
- net D1: now also U166.120 (PT53A)
- net D2: now also U166.119 (PT53B)
- net D3: now also U166.118 (PT56A)
- net D4: now also U166.116 (PT58A)
- net D5: now also U166.117 (PT56B)
- net D6: now also U166.115 (PT58B)
- net D7: now also U166.114 (PT60A)
- net DONE: now also U166.56 (DONE)
- net GND: now also R23.2, R24.2, R25.2, R26.2, R29.1, U166.101 (GND), U166.123 (GND), U166.129 (GND), U166.131 (GND), U166.138 (GND), U166.15 (GND), U166.21 (GND), U166.42 (GND), U166.65 (GND), U166.75 (GND), U166.8 (GND), U166.85 (GND), U166.87 (GND)
- net INITN: now also U166.55 (INITN)
- net IO2: now also U166.77 (PR41A)
- net IO3: now also U166.74 (PR41C)
- net MCLK: now also U166.54 (CCLK)
- net MISO/D1: now also U166.78 (PR35D)
- net MOSI/D0: now also U166.79 (PR35B)
- net OE#: now also U166.128 (PT29A)
- net PROGRAMN: now also U166.57 (PROGRAMN)
- net RCK: now also U166.44 (PB4B)
- net RD#: now also U166.135 (PT13B)
- net RXF#: now also U166.136 (PT13A)
- net RXI: now also U166.113 (PT60B)
- net SCK: now also U166.41 (PB6B)
- net SI_T1: now also U166.1 (PL5C)
- net SI_T10: now also U166.11 (PL14C)
- net SI_T11: now also U166.12 (PL14B)
- net SI_T12: now also U166.13 (PL14D)
- net SI_T13: now also U166.14 (PL23D)
- net SI_T14: now also U166.18 (PL32B)
- net SI_T15: now also U166.26 (PL41C)
- net SI_T16: now also U166.27 (PL41D)
- net SI_T17: now also U166.31 (PL44C)
- net SI_T18: now also U166.30 (PL44B)
- net SI_T19: now also U166.33 (PL44D)
- net SI_T2: now also U166.2 (PL5D)
- net SI_T20: now also U166.35 (PL47B)
- net SI_T21: now also U166.46 (PB11A)
- net SI_T22: now also U166.45 (PB9A)
- net SI_T23: now also U166.37 (PL47C)
- net SI_T24: now also U166.47 (PB11B)
- net SI_T25: now also U166.49 (PB15A)
- net SI_T26: now also U166.50 (PB13B)
- net SI_T27: now also U166.51 (PB15B)
- net SI_T28: now also U166.52 (PL18A)
- net SI_T29: now also U166.71 (PR47A)
- net SI_T3: now also U166.3 (PL5B)
- net SI_T30: now also U166.72 (PR44C)
- net SI_T31: now also U166.73 (PR41D)
- net SI_T32: now also U166.76 (PR41B)
- net SI_T4: now also U166.4 (PL8A)
- net SI_T5: now also U166.5 (PL8C)
- net SI_T6: now also U166.24 (PL38A)
- net SI_T7: now also U166.25 (PL38B)
- net SI_T8: now also U166.6 (PL8B)
- net SI_T9: now also U166.10 (PL14A)
- net TCK: now also R29.2, U166.63 (TCK)
- net TDI: now also R28.1, U166.61 (TDI)
- net TDO: now also R30.2, U166.60 (TDO)
- net TMS: now also R27.1, U166.64 (TMS)
- net TXE#: now also U166.134 (PT15A)
- net TXO: now also U166.112 (PT62A)
- net WR#: now also U166.133 (PT15B)
- new net: D12.1 (K), R26.1
- new net: D9.1 (K), R23.1
- new net: D11.1 (K), R25.1
- new net: D10.1 (K), R24.1
- new net HEART: D9.2 (A), U166.111 (PT62B)
- new net LED1: D10.2 (A), U166.110 (PT67A)
- new net LED2: D11.2 (A), U166.108 (PR2B)
- new net LED3: D12.2 (A), U166.107 (PR2C)
- no-connect marks 4 -> 2
Other:
- moved on the sheet: C66, D1, D2, J1, J4, J6, J7, J8, R10, R11, R12, R13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

Commit message: added more connections
Parts:
- added J9: Slave, symbol Connector_Generic:Conn_02x13_Odd_Even
Connections:
- net TCK: now also J9.1 (Pin_1), J9.2 (Pin_2)
- net TDI: now also J9.6 (Pin_6)
- net TDO: now also J9.5 (Pin_5), J9.8 (Pin_8)
- net TMS: now also J9.3 (Pin_3), J9.4 (Pin_4)
- net RELAY_D4: now reaches U166.102 (PR8D)
- net RELAY_D4: now also J9.15 (Pin_15)
- net RELAY_D3: now reaches U166.103 (PR8B)
- net RELAY_D3: now also J9.13 (Pin_13)
- net RELAY_D2: now reaches U166.104 (PR8C)
- net RELAY_D2: now also J9.11 (Pin_11)
- net RELAY_D1: now reaches U166.105 (PR8A)
- net RELAY_D1: now also J9.9 (Pin_9)
- net RELAY_D0: now reaches U166.106 (PR2D)
- net RELAY_D0: now also J9.7 (Pin_7)
- net RELAY_D7: now reaches U166.97 (PR14B)
- net RELAY_D7: now also J9.21 (Pin_21)
- net RELAY_D6: now reaches U166.98 (PR14C)
- net RELAY_D6: now also J9.19 (Pin_19)
- net RELAY_D5: now reaches U166.99 (PR14A)
- net RELAY_D5: now also J9.17 (Pin_17)
Other:
- note added: "LEFT SIDE IS FROM MASTER ECP AND RIGHT SLAVE ECP. NOTE: THE TDO CONNECTION GOES OUT FROM THE MASTER THEN GOES INTO SLAVE'S TDI THEN TDO GOES OUT FROM SLAVE TO THE FT2232H"
- moved on the sheet: D10, D11, D12, D3, D4, D5, D6, D7, D8, D9, J1, R20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
