File: hardware/projects/fpgapcb/.history/Transducer.kicad_sch (KiCad schematic)
At the start: 15 parts, among them U1 74HC595D, U3 MIC4127YML-TR, U4 MIC4127YML-TR, U6 MIC4127YML-TR

Commit message: not sure
Connections:
- net RCK renamed ARRAY-RCK
- net SCK renamed ARRAY-SCK
- net SI_T1 renamed ARRAY-SI_T1
Changed lines of the file:
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@@
 		)
 	)
-	(global_label "RCK"
+	(global_label "ARRAY-RCK"
 		(shape input)
 		(at 71.12 39.37 0)
@@
 		)
 	)
-	(global_label "SI_T1"
+	(global_label "ARRAY-SI_T1"
 		(shape input)
 		(at 77.47 25.4 90)
@@
 		)
 		(property "Intersheetrefs" "${INTERSHEET_REFS}"
-			(at 77.47 19.0449 90)
+			(at 77.47 13.1423 90)
 			(hide yes)
 			(show_name no)
@@
 		)
 	)
-	(global_label "SCK"
+	(global_label "ARRAY-SCK"
 		(shape input)
 		(at 71.12 36.83 0)
@@
 		)
 		(property "Intersheetrefs" "${INTERSHEET_REFS}"
-			(at 76.5075 36.83 0)
+			(at 82.4101 36.83 0)
 			(hide yes)
 			(show_name no)
