File: hardware/projects/fpgapcb/.history/Transducer15.kicad_sch (KiCad schematic)
At the start: 15 parts, among them U76 74HC595D, U77 MIC4127YML-TR, U78 MIC4127YML-TR, U79 MIC4127YML-TR, U80 MIC4127YML-TR

Commit message: not sure
Connections:
- net RCK renamed ARRAY-RCK
- net SCK renamed ARRAY-SCK
- net SI_T15 renamed ARRAY-SI_T15
Changed lines of the file:
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@@
 		)
 	)
-	(global_label "RCK"
+	(global_label "ARRAY-RCK"
 		(shape input)
 		(at 80.01 39.37 0)
@@
 		)
 	)
-	(global_label "SI_T15"
+	(global_label "ARRAY-SI_T15"
 		(shape input)
-		(at 86.36 24.13 90)
+		(at 86.36 29.21 90)
 		(fields_autoplaced yes)
 		(effects
@@
 		)
 		(property "Intersheetrefs" "${INTERSHEET_REFS}"
-			(at 86.36 14.9763 90)
+			(at 86.36 12.6781 90)
 			(hide yes)
 			(show_name no)
@@
 		)
 	)
-	(global_label "SCK"
+	(global_label "ARRAY-SCK"
 		(shape input)
 		(at 80.01 36.83 0)
@@
 		)
 		(property "Intersheetrefs" "${INTERSHEET_REFS}"
-			(at 85.3975 36.83 0)
+			(at 91.3001 36.83 0)
 			(hide yes)
 			(show_name no)
