File: hardware/projects/fpgapcb/.history/Transducer20.kicad_sch (KiCad schematic)
At the start: 15 parts, among them U101 74HC595D, U102 MIC4127YML-TR, U103 MIC4127YML-TR, U104 MIC4127YML-TR, U105 MIC4127YML-TR

Commit message: not sure
Connections:
- net RCK renamed ARRAY-RCK
- net SCK renamed ARRAY-SCK
- net SI_T20 renamed ARRAY-SI_T20
Changed lines of the file:
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@@
 		)
 	)
-	(global_label "SI_T20"
+	(global_label "ARRAY-SI_T20"
 		(shape input)
-		(at 83.82 24.13 90)
+		(at 83.82 29.21 90)
 		(fields_autoplaced yes)
 		(effects
@@
 		)
 		(property "Intersheetrefs" "${INTERSHEET_REFS}"
-			(at 83.82 14.9763 90)
+			(at 83.82 12.6781 90)
 			(hide yes)
 			(show_name no)
@@
 		)
 	)
-	(global_label "RCK"
+	(global_label "ARRAY-RCK"
 		(shape input)
 		(at 77.47 38.1 0)
@@
 		)
 	)
-	(global_label "SCK"
+	(global_label "ARRAY-SCK"
 		(shape input)
 		(at 77.47 35.56 0)
@@
 		)
 		(property "Intersheetrefs" "${INTERSHEET_REFS}"
-			(at 82.8575 35.56 0)
+			(at 88.7601 35.56 0)
 			(hide yes)
 			(show_name no)
