File: hardware/projects/fpgapcb/.history/Transducer21.kicad_sch (KiCad schematic)
At the start: 15 parts, among them U106 74HC595D, U107 MIC4127YML-TR, U108 MIC4127YML-TR, U109 MIC4127YML-TR, U110 MIC4127YML-TR

Commit message: not sure
Connections:
- net RCK renamed ARRAY-RCK
- net SCK renamed ARRAY-SCK
- net SI_T21 renamed ARRAY-SI_T21
Changed lines of the file:
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@@
 		)
 	)
-	(global_label "SCK"
+	(global_label "ARRAY-SCK"
 		(shape input)
 		(at 80.01 38.1 0)
@@
 		)
 		(property "Intersheetrefs" "${INTERSHEET_REFS}"
-			(at 85.3975 38.1 0)
+			(at 91.3001 38.1 0)
 			(hide yes)
 			(show_name no)
@@
 		)
 	)
-	(global_label "RCK"
+	(global_label "ARRAY-RCK"
 		(shape input)
 		(at 80.01 40.64 0)
@@
 		)
 	)
-	(global_label "SI_T21"
+	(global_label "ARRAY-SI_T21"
 		(shape input)
-		(at 86.36 26.67 90)
+		(at 86.36 29.21 90)
 		(fields_autoplaced yes)
 		(effects
@@
 		)
 		(property "Intersheetrefs" "${INTERSHEET_REFS}"
-			(at 86.36 17.5163 90)
+			(at 86.36 12.6781 90)
 			(hide yes)
 			(show_name no)
