File: hardware/projects/fpgapcb/.history/Transducer25.kicad_sch (KiCad schematic)
At the start: 15 parts, among them U126 74HC595D, U127 MIC4127YML-TR, U128 MIC4127YML-TR, U129 MIC4127YML-TR, U130 MIC4127YML-TR

Commit message: not sure
Connections:
- net RCK renamed ARRAY-RCK
- net SCK renamed ARRAY-SCK
- net SI_T25 renamed ARRAY-SI_T25
Changed lines of the file:
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@@
 		)
 	)
-	(global_label "RCK"
+	(global_label "ARRAY-RCK"
 		(shape input)
 		(at 85.09 39.37 0)
@@
 		)
 	)
-	(global_label "SI_T25"
+	(global_label "ARRAY-SI_T25"
 		(shape input)
-		(at 91.44 26.67 90)
+		(at 91.44 30.48 90)
 		(fields_autoplaced yes)
 		(effects
@@
 		)
 		(property "Intersheetrefs" "${INTERSHEET_REFS}"
-			(at 91.44 17.5163 90)
+			(at 91.44 13.9481 90)
 			(hide yes)
 			(show_name no)
@@
 		)
 	)
-	(global_label "SCK"
+	(global_label "ARRAY-SCK"
 		(shape input)
 		(at 85.09 36.83 0)
@@
 		)
 		(property "Intersheetrefs" "${INTERSHEET_REFS}"
-			(at 90.4775 36.83 0)
+			(at 96.3801 36.83 0)
 			(hide yes)
 			(show_name no)
