File: hardware/projects/fpgapcb/.history/Transducer29.kicad_sch (KiCad schematic)
At the start: 15 parts, among them U146 74HC595D, U147 MIC4127YML-TR, U148 MIC4127YML-TR, U149 MIC4127YML-TR, U150 MIC4127YML-TR

Commit message: not sure
Connections:
- net RCK renamed ARRAY-RCK
- net SCK renamed ARRAY-SCK
- net SI_T29 renamed ARRAY-SI_T29
Changed lines of the file:
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@@
 		)
 	)
-	(global_label "RCK"
+	(global_label "ARRAY-RCK"
 		(shape input)
 		(at 81.28 40.64 0)
@@
 		)
 	)
-	(global_label "SI_T29"
+	(global_label "ARRAY-SI_T29"
 		(shape input)
-		(at 87.63 26.67 90)
+		(at 87.63 30.48 90)
 		(fields_autoplaced yes)
 		(effects
@@
 		)
 		(property "Intersheetrefs" "${INTERSHEET_REFS}"
-			(at 87.63 17.5163 90)
+			(at 87.63 13.9481 90)
 			(hide yes)
 			(show_name no)
@@
 		)
 	)
-	(global_label "SCK"
+	(global_label "ARRAY-SCK"
 		(shape input)
 		(at 81.28 38.1 0)
@@
 		)
 		(property "Intersheetrefs" "${INTERSHEET_REFS}"
-			(at 86.6675 38.1 0)
+			(at 92.5701 38.1 0)
 			(hide yes)
 			(show_name no)
