File: hardware/projects/fpgapcb/.history/Transducer3.kicad_sch (KiCad schematic)
At the start: 15 parts, among them U16 74HC595D, U17 MIC4127YML-TR, U18 MIC4127YML-TR, U19 MIC4127YML-TR, U20 MIC4127YML-TR

Commit message: not sure
Connections:
- net RCK renamed ARRAY-RCK
- net SCK renamed ARRAY-SCK
- net SI_T3 renamed ARRAY-SI_T3
Changed lines of the file:
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@@
 	(wire
 		(pts
-			(xy 83.82 31.75) (xy 83.82 25.4)
+			(xy 83.82 31.75) (xy 83.82 29.21)
 		)
 		(stroke
@@
 		)
 	)
-	(global_label "SI_T3"
+	(global_label "ARRAY-SI_T3"
 		(shape input)
-		(at 83.82 25.4 90)
+		(at 83.82 29.21 90)
 		(fields_autoplaced yes)
 		(effects
@@
 		)
 		(property "Intersheetrefs" "${INTERSHEET_REFS}"
-			(at 83.82 17.4558 90)
+			(at 83.82 13.8876 90)
 			(hide yes)
 			(show_name no)
@@
 		)
 	)
-	(global_label "SCK"
+	(global_label "ARRAY-SCK"
 		(shape input)
 		(at 77.47 36.83 0)
@@
 		)
 		(property "Intersheetrefs" "${INTERSHEET_REFS}"
-			(at 82.8575 36.83 0)
+			(at 88.7601 36.83 0)
 			(hide yes)
 			(show_name no)
@@
 		)
 	)
-	(global_label "RCK"
+	(global_label "ARRAY-RCK"
 		(shape input)
 		(at 77.47 39.37 0)
