File: hardware/projects/fpgapcb/.history/Transducer31.kicad_sch (KiCad schematic)
At the start: 15 parts, among them U156 74HC595D, U157 MIC4127YML-TR, U158 MIC4127YML-TR, U159 MIC4127YML-TR, U160 MIC4127YML-TR

Commit message: not sure
Connections:
- net RCK renamed ARRAY-RCK
- net SCK renamed ARRAY-SCK
- net SI_T31 renamed ARRAY-SI_T31
Changed lines of the file:
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@@
 		)
 	)
-	(global_label "RCK"
+	(global_label "ARRAY-RCK"
 		(shape input)
 		(at 74.93 38.1 0)
@@
 		)
 	)
-	(global_label "SCK"
+	(global_label "ARRAY-SCK"
 		(shape input)
 		(at 74.93 35.56 0)
@@
 		)
 		(property "Intersheetrefs" "${INTERSHEET_REFS}"
-			(at 80.3175 35.56 0)
+			(at 86.2201 35.56 0)
 			(hide yes)
 			(show_name no)
@@
 		)
 	)
-	(global_label "SI_T31"
+	(global_label "ARRAY-SI_T31"
 		(shape input)
-		(at 81.28 25.4 90)
+		(at 81.28 29.21 90)
 		(fields_autoplaced yes)
 		(effects
@@
 		)
 		(property "Intersheetrefs" "${INTERSHEET_REFS}"
-			(at 81.28 16.2463 90)
+			(at 81.28 12.6781 90)
 			(hide yes)
 			(show_name no)
