File: hardware/projects/fpgapcb/.history/Transducer5.kicad_sch (KiCad schematic)
At the start: 15 parts, among them U26 74HC595D, U27 MIC4127YML-TR, U28 MIC4127YML-TR, U29 MIC4127YML-TR, U30 MIC4127YML-TR

Commit message: not sure
Connections:
- net RCK renamed ARRAY-RCK
- net SCK renamed ARRAY-SCK
- net SI_T5 renamed ARRAY-SI_T5
Changed lines of the file:
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@@
 		)
 	)
-	(global_label "SCK"
+	(global_label "ARRAY-SCK"
 		(shape input)
 		(at 74.93 38.1 0)
@@
 		)
 		(property "Intersheetrefs" "${INTERSHEET_REFS}"
-			(at 80.3175 38.1 0)
+			(at 86.2201 38.1 0)
 			(hide yes)
 			(show_name no)
@@
 		)
 	)
-	(global_label "SI_T5"
+	(global_label "ARRAY-SI_T5"
 		(shape input)
 		(at 81.28 27.94 90)
@@
 		)
 		(property "Intersheetrefs" "${INTERSHEET_REFS}"
-			(at 81.28 19.9958 90)
+			(at 81.28 12.6176 90)
 			(hide yes)
 			(show_name no)
@@
 		)
 	)
-	(global_label "RCK"
+	(global_label "ARRAY-RCK"
 		(shape input)
 		(at 74.93 40.64 0)
