File: hardware/projects/fpgapcb/.history/Transducer6.kicad_sch (KiCad schematic)
At the start: 15 parts, among them U31 74HC595D, U32 MIC4127YML-TR, U33 MIC4127YML-TR, U34 MIC4127YML-TR, U35 MIC4127YML-TR

Commit message: not sure
Connections:
- net RCK renamed ARRAY-RCK
- net SCK renamed ARRAY-SCK
- net SI_T6 renamed ARRAY-SI_T6
Changed lines of the file:
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@@
 	(wire
 		(pts
-			(xy 86.36 31.75) (xy 86.36 25.4)
+			(xy 86.36 31.75) (xy 86.36 27.94)
 		)
 		(stroke
@@
 		)
 	)
-	(global_label "SI_T6"
+	(global_label "ARRAY-SI_T6"
 		(shape input)
-		(at 86.36 25.4 90)
+		(at 86.36 27.94 90)
 		(fields_autoplaced yes)
 		(effects
@@
 		)
 		(property "Intersheetrefs" "${INTERSHEET_REFS}"
-			(at 86.36 17.4558 90)
+			(at 86.36 12.6176 90)
 			(hide yes)
 			(show_name no)
@@
 		)
 	)
-	(global_label "SCK"
+	(global_label "ARRAY-SCK"
 		(shape input)
 		(at 80.01 36.83 0)
@@
 		)
 		(property "Intersheetrefs" "${INTERSHEET_REFS}"
-			(at 85.3975 36.83 0)
+			(at 91.3001 36.83 0)
 			(hide yes)
 			(show_name no)
@@
 		)
 	)
-	(global_label "RCK"
+	(global_label "ARRAY-RCK"
 		(shape input)
 		(at 80.01 39.37 0)
