File: hardware/projects/fpgapcb/.history/Transducer8.kicad_sch (KiCad schematic)
At the start: 15 parts, among them U41 74HC595D, U42 MIC4127YML-TR, U43 MIC4127YML-TR, U44 MIC4127YML-TR, U45 MIC4127YML-TR

Commit message: not sure
Connections:
- net RCK renamed ARRAY-RCK
- net SCK renamed ARRAY-SCK
- net SI_T8 renamed ARRAY-SI_T8
Changed lines of the file:
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@@
 	(wire
 		(pts
-			(xy 81.28 31.75) (xy 81.28 25.4)
+			(xy 81.28 31.75) (xy 81.28 27.94)
 		)
 		(stroke
@@
 		)
 	)
-	(global_label "SCK"
+	(global_label "ARRAY-SCK"
 		(shape input)
 		(at 76.2 36.83 0)
@@
 		)
 		(property "Intersheetrefs" "${INTERSHEET_REFS}"
-			(at 81.5875 36.83 0)
+			(at 87.4901 36.83 0)
 			(hide yes)
 			(show_name no)
@@
 		)
 	)
-	(global_label "SI_T8"
+	(global_label "ARRAY-SI_T8"
 		(shape input)
-		(at 81.28 25.4 90)
+		(at 81.28 27.94 90)
 		(fields_autoplaced yes)
 		(effects
@@
 		)
 		(property "Intersheetrefs" "${INTERSHEET_REFS}"
-			(at 81.28 17.4558 90)
+			(at 81.28 12.6176 90)
 			(hide yes)
 			(show_name no)
@@
 		)
 	)
-	(global_label "RCK"
+	(global_label "ARRAY-RCK"
 		(shape input)
 		(at 76.2 39.37 0)
