File: hardware/projects/fpgapcb/.history/Transducer9.kicad_sch (KiCad schematic)
At the start: 15 parts, among them U46 74HC595D, U47 MIC4127YML-TR, U48 MIC4127YML-TR, U49 MIC4127YML-TR, U50 MIC4127YML-TR

Commit message: not sure
Connections:
- net RCK renamed ARRAY-RCK
- net SCK renamed ARRAY-SCK
- net SI_T9 renamed ARRAY-SI_T9
Changed lines of the file:
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@@
 	(wire
 		(pts
-			(xy 85.09 30.48) (xy 85.09 24.13)
+			(xy 85.09 30.48) (xy 85.09 27.94)
 		)
 		(stroke
@@
 		)
 	)
-	(global_label "SI_T9"
+	(global_label "ARRAY-SI_T9"
 		(shape input)
-		(at 85.09 24.13 90)
+		(at 85.09 27.94 90)
 		(fields_autoplaced yes)
 		(effects
@@
 		)
 		(property "Intersheetrefs" "${INTERSHEET_REFS}"
-			(at 85.09 16.1858 90)
+			(at 85.09 12.6176 90)
 			(hide yes)
 			(show_name no)
@@
 		)
 	)
-	(global_label "SCK"
+	(global_label "ARRAY-SCK"
 		(shape input)
 		(at 80.01 35.56 0)
@@
 		)
 		(property "Intersheetrefs" "${INTERSHEET_REFS}"
-			(at 85.3975 35.56 0)
+			(at 91.3001 35.56 0)
 			(hide yes)
 			(show_name no)
@@
 		)
 	)
-	(global_label "RCK"
+	(global_label "ARRAY-RCK"
 		(shape input)
 		(at 80.01 38.1 0)
