File: hardware/projects/fpgapcb/.history/ch340c.kicad_sch (KiCad schematic)
At the start: 2 parts, among them J1 Conn_01x06, U2 CH340C

Commit message: power good
Changed lines of the file:
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@@
 	(generator_version "10.0")
 	(paper "A4")
-	(text_box "CH340C"
+	(text_box "CH340C debug"
 		(exclude_from_sim no)
 		(at 111.76 45.72 0)

Commit message: not sure
Connections:
- net RXI renamed DEBUG-RXI
- net TXO renamed DEBUG-TXO
Changed lines of the file:
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@@
 		)
 	)
-	(global_label "TXO"
+	(global_label "DEBUG-TXO"
 		(shape input)
 		(at 154.94 55.88 0)
@@
 		)
 		(property "Intersheetrefs" "${INTERSHEET_REFS}"
-			(at 161.4328 55.88 0)
+			(at 169.2947 55.88 0)
 			(hide yes)
 			(show_name no)
@@
 		)
 	)
-	(global_label "RXI"
+	(global_label "DEBUG-RXI"
 		(shape input)
 		(at 154.94 58.42 0)
@@
 		)
 		(property "Intersheetrefs" "${INTERSHEET_REFS}"
-			(at 161.0095 58.42 0)
+			(at 168.8714 58.42 0)
 			(hide yes)
 			(show_name no)
@@
 		)
 	)
-	(global_label "TXO"
+	(global_label "DEBUG-TXO"
 		(shape input)
 		(at 151.13 114.3 0)
@@
 		)
 		(property "Intersheetrefs" "${INTERSHEET_REFS}"
-			(at 157.6228 114.3 0)
+			(at 165.4847 114.3 0)
 			(hide yes)
 			(show_name no)
@@
 		)
 	)
-	(global_label "RXI"
+	(global_label "DEBUG-RXI"
 		(shape input)
 		(at 151.13 111.76 0)
@@
 		)
 		(property "Intersheetrefs" "${INTERSHEET_REFS}"
-			(at 157.1995 111.76 0)
+			(at 165.0614 111.76 0)
 			(hide yes)
 			(show_name no)

Commit message: added 5v & trigger notes
Parts:
- renumbered J1 to J4
Changed lines of the file:
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@@
 		(in_pos_files yes)
 		(dnp no)
-		(property "Reference" "#PWR0518"
+		(property "Reference" "#PWR0519"
 			(at 137.16 93.98 0)
 			(hide yes)
@@
 		)
 		(instances
-			(project "link"
-				(path "/9c5ef320-ed14-4fbf-afec-63494d4e827d"
-					(reference "#PWR0518")
+			(project "main_fpga_board_link"
+				(path "/de89ff7a-3cfc-4f81-afc2-8cb9be17c69a/adfed331-e330-4f8f-b1fa-9964b9752d9b"
+					(reference "#PWR0519")
 					(unit 1)
 				)
@@
 		(dnp no)
 		(fields_autoplaced yes)
-		(property "Reference" "J1"
+		(property "Reference" "J4"
 			(at 137.16 97.79 0)
 			(show_name no)
@@
 		)
 		(instances
-			(project "link"
-				(path "/9c5ef320-ed14-4fbf-afec-63494d4e827d"
-					(reference "J1")
+			(project "main_fpga_board_link"
+				(path "/de89ff7a-3cfc-4f81-afc2-8cb9be17c69a/adfed331-e330-4f8f-b1fa-9964b9752d9b"
+					(reference "J4")
 					(unit 1)
 				)
@@
 		)
 		(instances
-			(project "link"
-				(path "/9c5ef320-ed14-4fbf-afec-63494d4e827d"
+			(project "main_fpga_board_link"
+				(path "/de89ff7a-3cfc-4f81-afc2-8cb9be17c69a/adfed331-e330-4f8f-b1fa-9964b9752d9b"
 					(reference "U2")
 					(unit 1)
@@
 		(in_pos_files yes)
 		(dnp no)
-		(property "Reference" "#PWR0517"
+		(property "Reference" "#PWR0520"
 			(at 151.13 127 0)
 			(hide yes)
@@
 		)
 		(instances
-			(project "link"
-				(path "/9c5ef320-ed14-4fbf-afec-63494d4e827d"
-					(reference "#PWR0517")
+			(project "main_fpga_board_link"
+				(path "/de89ff7a-3cfc-4f81-afc2-8cb9be17c69a/adfed331-e330-4f8f-b1fa-9964b9752d9b"
+					(reference "#PWR0520")
 					(unit 1)
 				)
@@
 		)
 	)
-	(sheet_instances
-		(path "/"
-			(page "5")
-		)
-	)
