File: hardware/projects/arraypcb/Transducer13.kicad_sch (KiCad schematic)
At the start: 15 parts, among them U66 74HC595D, U67 MIC4127YML-TR, U68 MIC4127YML-TR, U69 MIC4127YML-TR, U70 MIC4127YML-TR

Commit message: moved slave d7+- to bank 7 and adjusted ftdi-0 accordingly; replaced all +5v rails to +20v
Connections:
- net +5V renamed +20V
Changed lines of the file:
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@@
 			)
 		)
-		(property "Value" "+5V"
+		(property "Value" "+20V"
 			(at 264.16 26.67 0)
 			(show_name no)
@@
 			)
 		)
-		(property "Value" "+5V"
+		(property "Value" "+20V"
 			(at 162.56 16.51 0)
 			(show_name no)
