File: hardware/projects/arraypcb/Transducer27.kicad_sch (KiCad schematic)
At the start: 15 parts, among them U136 74HC595D, U137 MIC4127YML-TR, U138 MIC4127YML-TR, U139 MIC4127YML-TR, U140 MIC4127YML-TR

Commit message: moved slave d7+- to bank 7 and adjusted ftdi-0 accordingly; replaced all +5v rails to +20v
Connections:
- net +5V renamed +20V
Changed lines of the file:
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@@
 			)
 		)
-		(property "Value" "+5V"
+		(property "Value" "+20V"
 			(at 171.45 17.78 0)
 			(show_name no)
@@
 			)
 		)
-		(property "Value" "+5V"
+		(property "Value" "+20V"
 			(at 273.05 27.94 0)
 			(show_name no)
