File: hardware/projects/arraypcb/Transducer28.kicad_sch (KiCad schematic)
At the start: 15 parts, among them U141 74HC595D, U142 MIC4127YML-TR, U143 MIC4127YML-TR, U144 MIC4127YML-TR, U145 MIC4127YML-TR

Commit message: moved slave d7+- to bank 7 and adjusted ftdi-0 accordingly; replaced all +5v rails to +20v
Connections:
- net +5V renamed +20V
Changed lines of the file:
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@@
 			)
 		)
-		(property "Value" "+5V"
+		(property "Value" "+20V"
 			(at 166.37 15.24 0)
 			(show_name no)
@@
 			)
 		)
-		(property "Value" "+5V"
+		(property "Value" "+20V"
 			(at 267.97 25.4 0)
 			(show_name no)
