File: hardware/projects/arraypcb/Transducer29.kicad_sch (KiCad schematic)
At the start: 15 parts, among them U146 74HC595D, U147 MIC4127YML-TR, U148 MIC4127YML-TR, U149 MIC4127YML-TR, U150 MIC4127YML-TR

Commit message: moved slave d7+- to bank 7 and adjusted ftdi-0 accordingly; replaced all +5v rails to +20v
Connections:
- net +5V renamed +20V
Changed lines of the file:
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@@
 			)
 		)
-		(property "Value" "+5V"
+		(property "Value" "+20V"
 			(at 167.64 19.05 0)
 			(show_name no)
@@
 			)
 		)
-		(property "Value" "+5V"
+		(property "Value" "+20V"
 			(at 269.24 29.21 0)
 			(show_name no)
