File: hardware/projects/fpgapcb/Decoupling_caps.kicad_sch (KiCad schematic)
At the start: 27 parts

Commit message: added testpoints; schematic tidyness; removed data & sync to give way for the connection between two control boards
Parts:
- renumbered C15 to C100, C17 to C101, C19 to C102, C21 to C103, C24 to C104, C25 to C105, C26 to C106, C27 to C107, C8 to C108, C4 to C65, C2 to C84, C3 to C85, C6 to C86, C10 to C87, C12 to C88, C14 to C89, C16 to C90, C18 to C91, C20 to C92, C22 to C93, C23 to C94, C5 to C95, C7 to C96, C9 to C97, C11 to C98, C13 to C99
