File: hardware/projects/fpgapcb/power.kicad_sch (KiCad schematic)
At the start: 24 parts, among them J4 Screw_Terminal_01x02, U10 TLV62569DBV, U8 TPS54302, U9 TLV62569DBV

Commit message: added 5v & trigger notes
Parts:
- added C75: 10μF, Capacitor_SMD:C_0805_2012Metric, symbol Device:C_Small
- added C76, C80: 0.1μF, Capacitor_SMD:C_0805_2012Metric, symbol Device:C_Small
- added C77, C78: 22μF, Capacitor_SMD:C_0805_2012Metric, symbol Device:C_Small
- added C79: 75pF, Capacitor_SMD:C_0805_2012Metric, symbol Device:C_Small
- added L4: 10μH, Inductor_SMD:L_Bourns_SRN6045TA, symbol Device:L
- added R28: 105k, Resistor_SMD:R_0805_2012Metric, symbol Device:R_Small_US
- added R30: 511k, Resistor_SMD:R_0805_2012Metric, symbol Device:R_Small_US
- added R34: 49.9, Resistor_SMD:R_0805_2012Metric, symbol Device:R_Small_US
- added R35: 100k, Resistor_SMD:R_0805_2012Metric, symbol Device:R_Small_US
- added R36: 13.3k, Resistor_SMD:R_0805_2012Metric, symbol Device:R_Small_US
- added U11: TPS54302, Package_TO_SOT_SMD:SOT-23-6, symbol Regulator_Switching:TPS54302
Connections:
- net 12V: now also C75.1, C80.1, R30.1, U11.3 (VIN); no longer U8.5 (EN)
- net GND: now also C75.2, C77.2, C78.2, C80.2, R28.2, R36.2, U11.1 (GND)
- new net: C76.1, U11.6 (BOOT)
- new net: C76.2, L4.1, U11.2 (SW)
- new net: C79.1, R34.2, R35.1
- new net: R28.1, R30.2, U11.5 (EN)
- new net: C79.2, R35.2, R36.1, U11.4 (FB)
- new net 5V: C77.1, C78.1, L4.2, R34.1
- no-connect marks 0 -> 1
Other:
- moved on the sheet: C66, C67, C68, C69, C70, C71, C72, C73, C74, D1, D2, J4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

Commit message: added testpoints; schematic tidyness; removed data & sync to give way for the connection between two control boards
Other:
- sheet FPGA_POWER renamed Decoupling caps
- sheet Decoupling caps: file FPGA_POWER.kicad_sch -> Decoupling_caps.kicad_sch
Changed lines of the file:
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@@
 			(color 0 0 0 0)
 		)
-		(property "Sheetname" "FPGA_POWER"
+		(property "Sheetname" "Decoupling caps"
 			(at 212.09 116.1284 0)
 			(show_name no)
@@
 			)
 		)
-		(property "Sheetfile" "FPGA_POWER.kicad_sch"
+		(property "Sheetfile" "Decoupling_caps.kicad_sch"
 			(at 212.09 145.3646 0)
 			(show_name no)

Commit message: slave schematic added
Parts:
- renumbered C70 to C109, C74 to C110, C66 to C111, C72 to C112, C68 to C113, C69 to C114, C75 to C115, C80 to C116, C76 to C117, C77 to C118, C78 to C119, C79 to C120, C67 to C81, C73 to C82, C71 to C83, D1 to D23, D2 to D24, J4 to J15, L3 to L5, L2 to L6, L1 to L7, L4 to L8, R18 to R66, R19 to R67, R17 to R68, R16 to R69, R14 to R70, R15 to R71, R30 to R72, R28 to R73, R34 to R74, R35 to R75, R36 to R76, U10 to U13, U8 to U14, U9 to U15, U11 to U16
